File: pcbs/kicad/zuko-teensy-motor-controller/zuko-teensy-motor-controller.kicad_pcb (KiCad board)
At the start: 2 copper layers, 2 parts, among them J1 Conn_01x03, U1 Teensy4.0

Commit message: pcb update
Parts:
- added C1: 2200uF, Capacitor_THT:CP_Radial_D10.0mm_P5.00mm, F.Cu at (122.1, 76.2)
- added C2: 2200uF, Capacitor_THT:CP_Radial_D10.0mm_P5.00mm, F.Cu at (99.2, 91.4)
- added C3: 2200uF, Capacitor_THT:CP_Radial_D10.0mm_P5.00mm, F.Cu at (99.8, 76.3)
- added C4: 2200uF, Capacitor_THT:CP_Radial_D10.0mm_P5.00mm, F.Cu at (122.1, 91.4)
- added J10: Conn_01x03, Connector_PinHeader_2.54mm:PinHeader_1x03_P2.54mm_Vertical, F.Cu at (94.0, 73.7)
- added J11: Conn_01x03, Connector_PinHeader_2.54mm:PinHeader_1x03_P2.54mm_Vertical, F.Cu at (110.5, 73.7)
- added J12: Conn_01x03, Connector_PinHeader_2.54mm:PinHeader_1x03_P2.54mm_Vertical, F.Cu at (114.3, 73.7)
- added J13: Conn_01x03, Connector_PinHeader_2.54mm:PinHeader_1x03_P2.54mm_Vertical, F.Cu at (118.1, 73.7)
- added J14: Conn_01x02, Connector_PinHeader_2.54mm:PinHeader_1x02_P2.54mm_Vertical, F.Cu at (121.9, 39.4)
- added J15: Conn_01x02, Connector_PinHeader_2.54mm:PinHeader_1x02_P2.54mm_Vertical, F.Cu at (61.0, 55.9)
- added J16: Conn_01x02, Connector_PinHeader_2.54mm:PinHeader_1x02_P2.54mm_Vertical, F.Cu at (129.5, 39.4)
- added J17: Conn_01x03, Connector_PinHeader_2.54mm:PinHeader_1x03_P2.54mm_Vertical, F.Cu at (153.7, 88.9)
- added J18: Conn_01x03, Connector_PinHeader_2.54mm:PinHeader_1x03_P2.54mm_Vertical, F.Cu at (157.5, 88.9)
- added J19: Conn_01x02, Connector_PinHeader_2.54mm:PinHeader_1x02_P2.54mm_Vertical, F.Cu at (125.7, 39.4)
- added J2: Conn_01x03, Connector_PinHeader_2.54mm:PinHeader_1x03_P2.54mm_Vertical, F.Cu at (88.9, 88.9)
- added J20: Conn_01x02, Connector_PinHeader_2.54mm:PinHeader_1x02_P2.54mm_Vertical, F.Cu at (165.1, 83.8)
- added J21: Conn_01x02, Connector_PinHeader_2.54mm:PinHeader_1x02_P2.54mm_Vertical, F.Cu at (64.8, 55.9)
- added J22: Conn_01x03, Connector_PinHeader_2.54mm:PinHeader_1x03_P2.54mm_Vertical, F.Cu at (161.3, 88.9)
- added J23: Conn_01x03, Connector_PinHeader_2.54mm:PinHeader_1x03_P2.54mm_Vertical, F.Cu at (165.1, 88.9)
- added J24: Conn_01x04, Connector_PinHeader_2.54mm:PinHeader_1x04_P2.54mm_Vertical, F.Cu at (214.6, 85.1)
- added J25: Conn_01x03, Connector_PinHeader_2.54mm:PinHeader_1x03_P2.54mm_Vertical, F.Cu at (167.6, 71.1)
- added J26: Conn_01x03, Connector_PinHeader_2.54mm:PinHeader_1x03_P2.54mm_Vertical, F.Cu at (163.8, 71.1)
- added J27: Conn_01x04, Connector_PinHeader_2.54mm:PinHeader_1x04_P2.54mm_Vertical, F.Cu at (153.7, 55.9)
- added J28: Conn_01x04, Connector_PinHeader_2.54mm:PinHeader_1x04_P2.54mm_Vertical, F.Cu at (222.2, 85.1)
- added J29: Conn_01x04, Connector_PinHeader_2.54mm:PinHeader_1x04_P2.54mm_Vertical, F.Cu at (157.5, 55.9)
- added J3: Conn_01x03, Connector_PinHeader_2.54mm:PinHeader_1x03_P2.54mm_Vertical, F.Cu at (92.7, 88.9)
- added J30: Conn_01x04, Connector_PinHeader_2.54mm:PinHeader_1x04_P2.54mm_Vertical, F.Cu at (226.1, 85.1)
- added J31: Conn_01x04, Connector_PinHeader_2.54mm:PinHeader_1x04_P2.54mm_Vertical, F.Cu at (161.3, 55.9)
- added J32: Conn_01x04, Connector_PinHeader_2.54mm:PinHeader_1x04_P2.54mm_Vertical, F.Cu at (165.1, 55.9)
- added J33: Conn_01x04, Connector_PinHeader_2.54mm:PinHeader_1x04_P2.54mm_Vertical, F.Cu at (210.8, 85.1)
- added J4: Conn_01x02, Connector_AMASS:AMASS_XT60-F_1x02_P7.20mm_Vertical, F.Cu at (85.5, 57.1)
- added J5: Conn_01x03, Connector_PinHeader_2.54mm:PinHeader_1x03_P2.54mm_Vertical, F.Cu at (110.5, 88.9)
- added J6: Conn_01x03, Connector_PinHeader_2.54mm:PinHeader_1x03_P2.54mm_Vertical, F.Cu at (114.3, 88.9)
- added J7: Conn_01x03, Connector_PinHeader_2.54mm:PinHeader_1x03_P2.54mm_Vertical, F.Cu at (118.1, 88.9)
- added J8: Conn_01x03, Connector_PinHeader_2.54mm:PinHeader_1x03_P2.54mm_Vertical, F.Cu at (86.4, 73.7)
- added J9: Conn_01x03, Connector_PinHeader_2.54mm:PinHeader_1x03_P2.54mm_Vertical, F.Cu at (90.2, 73.7)
- added JP1: Jumper_3_Open, Connector_PinHeader_2.54mm:PinHeader_1x03_P2.54mm_Vertical, F.Cu at (153.7, 83.8)
- added Q1: BSS138, Package_TO_SOT_SMD:SOT-23, F.Cu at (229.5, 123.5)
- added Q2: BSS138, Package_TO_SOT_SMD:SOT-23, F.Cu at (229.5, 117.8)
- added R11: 10k, Resistor_SMD:R_1206_3216Metric_Pad1.30x1.75mm_HandSolder, F.Cu at (217.8, 109.0)
- added R12: 10k, Resistor_SMD:R_1206_3216Metric_Pad1.30x1.75mm_HandSolder, F.Cu at (164.9, 141.0)
- added R13: 10k, Resistor_SMD:R_1206_3216Metric_Pad1.30x1.75mm_HandSolder, F.Cu at (183.2, 140.6)
- added R14: 10k, Resistor_SMD:R_1206_3216Metric_Pad1.30x1.75mm_HandSolder, F.Cu at (159.0, 141.0)
- added U1: ACS712xLCTR-20A, Package_SO:SOIC-8_3.9x4.9mm_P1.27mm, F.Cu at (88.9, 66.0)
- moved J1 104.4 mm to (85.1, 88.9)
- moved U2 27.3 mm to (141.0, 71.1), turned to -90 degrees
- renumbered U1 to U2
Connections:
- J1 pad 1: unconnected-(J1-Pad1) -> M1
- J1 pad 2: unconnected-(J1-Pad2) -> +BATT
- J1 pad 3: unconnected-(J1-Pad3) -> GND
Other:
- board outline added: 100 x 45 mm
