File: pcbs/kicad/zuko-teensy-motor-controller/zuko-teensy-motor-controller.kicad_pcb (KiCad board)
At the start: 4 copper layers, 100 x 40 mm, 66 parts, among them J1 Conn_01x03, J10 Conn_01x03, J11 Conn_01x03, J12 Conn_01x03, J13 Conn_01x03, J14 Conn_01x02, J15 Conn_01x02, J16 Conn_01x02, J17 Conn_01x03, J18 Conn_01x03, J19 Conn_01x02, J2 Conn_01x03, J20 Conn_01x02, J21 Conn_01x02, J22 Conn_01x03, J23 Conn_01x02, J24 Conn_01x04, J25 Conn_01x03, J26 Conn_01x03, J27 Conn_01x04, J28 Conn_01x04, J29 Conn_01x04, J3 Conn_01x03, J30 Conn_01x04, J31 Conn_01x04, J32 Conn_01x04, J33 Conn_01x04, J34 Conn_01x02, J4 Conn_01x02, J5 Conn_01x03, J6 Conn_01x03, J7 Conn_01x03, J8 Conn_01x03, J9 Conn_01x03, Q1 BSS138, Q2 BSS138, U1 ACS712xLCTR-20A, U2 Teensy4.0, U3 ULN2003

Commit message: review file upload
Routing:
- net RX: track 13.6 -> 17.9 mm
- net Net-(J4-Pad1): track 55.7 -> 55.8 mm, vias 2 -> 5
Changed lines of the file:
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@@
     (property "Sheetname" "")
     (attr through_hole)
-    (fp_text reference "J4" (at 2.5 -4) (layer "F.SilkS")
+    (fp_text reference "J4" (at 2.5 -4) (layer "F.SilkS") hide
       (effects (font (size 1 1) (thickness 0.15)))
     )
-    (fp_text value "Conn_01x02" (at 2.5 4) (layer "F.Fab")
+    (fp_text value "Conn_01x02" (at 2.5 4) (layer "F.Fab") hide
       (effects (font (size 1 1) (thickness 0.15)))
     )
-    (fp_text user "+" (at 9 0) (layer "F.SilkS")
+    (fp_text user "+" (at 9 0) (layer "F.SilkS") hide
       (effects (font (size 1.5 1.5) (thickness 0.15)))
     )
-    (fp_text user "-" (at -4 0) (layer "F.SilkS")
+    (fp_text user "-" (at -4 0) (layer "F.SilkS") hide
       (effects (font (size 1.5 1.5) (thickness 0.15)))
     )
-    (fp_text user "${REFERENCE}" (at 2.5 0) (layer "F.Fab")
+    (fp_text user "${REFERENCE}" (at 2.5 0) (layer "F.Fab") hide
       (effects (font (size 1 1) (thickness 0.15)))
     )
@@
     (effects (font (size 2 2) (thickness 0.3)))
   )
+  (gr_text "+" (at 84.45 44.89 270) (layer "F.SilkS")
+    (effects (font (size 1.27 1.27) (thickness 0.2032)))
+  )
   (gr_text "GND\n" (at 133.52 50.7 270) (layer "F.SilkS")
     (effects (font (size 1.016 1.016) (thickness 0.2032)))
@@
     (effects (font (size 0.762 0.762) (thickness 0.1524)))
   )
+  (gr_text "-" (at 84.38 47.28) (layer "F.SilkS")
+    (effects (font (size 1.27 1.27) (thickness 0.2032)))
+  )
   (gr_text "3V3" (at 141.32 50.7 270) (layer "F.SilkS")
     (effects (font (size 1.016 1.016) (thickness 0.2032)))
@@
   (segment (start 113.566791 49.733209) (end 116.0984 47.2016) (width 0.3302) (layer "F.Cu") (net 32))
   (segment (start 113.5916 55.292) (end 113.566791 55.267191) (width 0.3302) (layer "F.Cu") (net 32))
+  (segment (start 111.138 59.86385) (end 112.2 60.92585) (width 0.3302) (layer "F.Cu") (net 33))
+  (segment (start 111.138 57.6254) (end 111.138 59.86385) (width 0.3302) (layer "F.Cu") (net 33))
   (segment (start 113.99 61.5) (end 114.01 61.52) (width 0.3302) (layer "F.Cu") (net 33))
   (segment (start 112.2 61.5) (end 113.99 61.5) (width 0.3302) (layer "F.Cu") (net 33))
+  (segment (start 112.2 60.92585) (end 112.2 61.5) (width 0.3302) (layer "F.Cu") (net 33))
   (via (at 114.01 61.52) (size 0.8) (drill 0.4) (layers "F.Cu" "B.Cu") (net 33))
   (segment (start 114.01 55.914798) (end 109.654602 51.5594) (width 0.3302) (layer "In1.Cu") (net 33))
@@
   (segment (start 69.56 49.89) (end 69.56 57.37) (width 2.5) (layer "F.Cu") (net 46))
   (segment (start 69.56 57.37) (end 69.48 57.45) (width 2.5) (layer "F.Cu") (net 46))
+  (via (at 69.52 53.29) (size 0.8) (drill 0.4) (layers "F.Cu" "B.Cu") (net 46))
+  (via (at 69.4 50.76) (size 0.8) (drill 0.4) (layers "F.Cu" "B.Cu") (net 46))
   (via (at 67.78 57.45) (size 0.8) (drill 0.4) (layers "F.Cu" "B.Cu") (net 46))
   (via (at 69.56 55.435) (size 0.8) (drill 0.4) (layers "F.Cu" "B.Cu") (net 46))
+  (via (at 70.6 48.89) (size 0.8) (drill 0.4) (layers "F.Cu" "B.Cu") (net 46))
   (segment (start 69.56 55.67) (end 67.78 57.45) (width 2.5) (layer "In1.Cu") (net 46))
-  (segment (start 69.56 50.5202) (end 69.56 55.435) (width 2.5) (layer "In1.Cu") (net 46))
-  (segment (start 73.36 46.7202) (end 69.56 50.5202) (width 2.5) (layer "In1.Cu") (net 46))
-  (segment (start 73.36 46.09) (end 73.36 46.7202) (width 2.5) (layer "In1.Cu") (net 46))
+  (segment (start 73.36 46.09) (end 73.31 46.09) (width 2.5) (layer "In1.Cu") (net 46))
+  (segment (start 69.56 49.84) (end 69.56 55.435) (width 2.5) (layer "In1.Cu") (net 46))
+  (segment (start 73.31 46.09) (end 69.56 49.84) (width 2.5) (layer "In1.Cu") (net 46))
   (segment (start 69.56 55.435) (end 69.56 55.67) (width 2.5) (layer "In1.Cu") (net 46))
-  (segment (start 73.36 46.7202) (end 73.36 46.09) (width 2.5) (layer "In2.Cu") (net 46))
+  (segment (start 69.59 49.79) (end 73.29 46.09) (width 2.5) (layer "In2.Cu") (net 46))
+  (segment (start 69.59 54.75987) (end 69.59 49.79) (width 2.5) (layer "In2.Cu") (net 46))
   (segment (start 69.62 55.61) (end 69.62 54.78987) (width 2.5) (layer "In2.Cu") (net 46))
-  (segment (start 67.78 57.45) (end 69.62 55.61) (width 2.5) (layer "In2.Cu") (net 46))
+  (segment (start 73.29 46.09) (end 73.36 46.09) (width 2.5) (layer "In2.Cu") (net 46))
   (segment (start 69.62 54.78987) (end 69.59 54.75987) (width 2.5) (layer "In2.Cu") (net 46))
-  (segment (start 69.59 50.4902) (end 73.36 46.7202) (width 2.5) (layer "In2.Cu") (net 46))
-  (segment (start 69.59 54.75987) (end 69.59 50.4902) (width 2.5) (layer "In2.Cu") (net 46))
-  (segment (start 69.6 50.38) (end 69.6 55.63) (width 2.5) (layer "B.Cu") (net 46))
-  (segment (start 73.36 46.62) (end 69.6 50.38) (width 2.5) (layer "B.Cu") (net 46))
-  (segment (start 73.36 46.09) (end 73.36 46.62) (width 2.5) (layer "B.Cu") (net 46))
+  (segment (start 67.78 57.45) (end 69.62 55.61) (width 2.5) (layer "In2.Cu") (net 46))
+  (segment (start 73.36 46.09) (end 73.36 46.13) (width 2.5) (layer "B.Cu") (net 46))
   (segment (start 69.6 55.63) (end 67.78 57.45) (width 2.5) (layer "B.Cu") (net 46))
+  (segment (start 73.36 46.13) (end 69.6 49.89) (width 2.5) (layer "B.Cu") (net 46))
+  (segment (start 69.6 49.89) (end 69.6 55.63) (width 2.5) (layer "B.Cu") (net 46))
   (segment (start 89.27498 54.76498) (end 89.22 54.71) (width 0.3302) (layer "F.Cu") (net 47))
   (segment (start 87.22 57.15) (end 89.27498 57.15) (width 0.3302) (layer "F.Cu") (net 47))
