File: pcbs/kicad/zuko-teensy-motor-controller/zuko-teensy-motor-controller.kicad_sch (KiCad schematic)
At the start: 44 parts, among them J1 Conn_01x03, J10 Conn_01x03, J11 Conn_01x03, J12 Conn_01x03, J13 Conn_01x03, J14 Conn_01x03, J15 Conn_01x03, J16 Conn_01x03, J17 Conn_01x03, J18 Conn_01x03, J19 Conn_01x04, J2 Conn_01x03, J20 Conn_01x04, J21 Conn_01x04, J22 Conn_01x04, J3 Conn_01x03, J4 Conn_01x03, J5 Conn_01x03, J6 Conn_01x03, J7 Conn_01x03, J8 Conn_01x03, J9 Conn_01x03, U1 Teensy4.0, U2 ULN2003

Commit message: pcb update
Parts:
- removed J4: Conn_01x03, Connector_PinHeader_2.54mm:PinHeader_1x03_P2.54mm_Vertical, symbol Connector_Generic:Conn_01x03
- removed JP1, JP2, JP4: Jumper_3_Open, symbol Jumper:Jumper_3_Open
- added C1, C2, C3, C4: 2200uF, Capacitor_THT:CP_Radial_D10.0mm_P5.00mm, symbol Device:C_Polarized_US
- added C5: 1nF, symbol Device:C
- added C6: 100nF, symbol Device:C
- added J13: Conn_01x03, Connector_PinHeader_2.54mm:PinHeader_1x03_P2.54mm_Vertical, symbol Connector_Generic:Conn_01x03
- added J14, J15, J16, J19, J20, J21: Conn_01x02, Connector_PinHeader_2.54mm:PinHeader_1x02_P2.54mm_Vertical, symbol Connector_Generic:Conn_01x02
- added J4: Conn_01x02, Connector_AMASS:AMASS_XT60-F_1x02_P7.20mm_Vertical, symbol Connector_Generic:Conn_01x02
- added R1, R2, R3: 10k, symbol Device:R_Small_US
- added R4: 20k, symbol Device:R_Small_US
- added U1: ACS712xLCTR-20A, Package_SO:SOIC-8_3.9x4.9mm_P1.27mm, symbol Sensor_Current:ACS712xLCTR-20A
- JP1: renamed from JP3; footprint (none) -> Connector_PinHeader_2.54mm:PinHeader_1x03_P2.54mm_Vertical
- gave numbers to parts that had none: 14
- renumbered J13 to J17, J14 to J18, J15 to J22, J16 to J23, J17 to J25, J18 to J26, J19 to J27, J20 to J29, J21 to J31, J22 to J32, R1 to R7, R2 to R8, U1 to U2, U2 to U3
Connections:
- net +5V: now also C6.1, J14.1 (Pin_1), J16.1 (Pin_1), J19.1 (Pin_1), R1.1, U1.8 (VCC)
- net +AUX: now also J20.1 (Pin_1)
- net +BATT: now also J1.2 (Pin_2), J10.2 (Pin_2), J11.2 (Pin_2), J12.2 (Pin_2), J2.2 (Pin_2), J3.2 (Pin_2), J5.2 (Pin_2), J6.2 (Pin_2), J7.2 (Pin_2), J8.2 (Pin_2), J9.2 (Pin_2), C1.1, C2.1, C3.1, C4.1, J13.2 (Pin_2), J15.1 (Pin_1), J21.1 (Pin_1), U1.3 (IP-), U1.4 (IP-); no longer J1.1 (Pin_1), J10.1 (Pin_1), J11.1 (Pin_1), J12.1 (Pin_1), J2.1 (Pin_1), J3.1 (Pin_1), J5.1 (Pin_1), J6.1 (Pin_1), J7.1 (Pin_1), J8.1 (Pin_1), J9.1 (Pin_1)
- net AUX_M1: no longer J18.2 (Pin_2), J22.2 (Pin_2), J23.2 (Pin_2)
- net GND: now also C1.2, C2.2, C3.2, C4.2, C5.2, C6.2, J13.3 (Pin_3), J14.2 (Pin_2), J15.2 (Pin_2), J16.2 (Pin_2), J19.2 (Pin_2), J20.2 (Pin_2), J21.2 (Pin_2), J4.2 (Pin_2), R3.2, R4.2, U1.5 (GND)
- net M1: now also J1.1 (Pin_1); no longer J1.2 (Pin_2)
- net M10: now also J11.1 (Pin_1); no longer J10.2 (Pin_2)
- net M11: now also J12.1 (Pin_1); no longer J11.2 (Pin_2)
- net M12: now also J13.1 (Pin_1); no longer J12.2 (Pin_2)
- net M2: now also J2.1 (Pin_1); no longer J2.2 (Pin_2)
- net M3: now also J3.1 (Pin_1); no longer J3.2 (Pin_2)
- net M4: now also J5.1 (Pin_1)
- net M5: now also J6.1 (Pin_1); no longer J5.2 (Pin_2)
- net M6: now also J7.1 (Pin_1); no longer J6.2 (Pin_2)
- net M7: now also J8.1 (Pin_1); no longer J7.2 (Pin_2)
- net M8: now also J9.1 (Pin_1); no longer J8.2 (Pin_2)
- net M9: now also J10.1 (Pin_1); no longer J9.2 (Pin_2)
- net SDA1: no longer J24.2 (Pin_2), R5.2
- net SDL1: no longer J24.3 (Pin_3), R6.2
- net at J22.1 (Pin_1), JP1.2 (C): now also J17.1 (Pin_1), J18.1 (Pin_1), J23.1 (Pin_1)
- new net: R2.1, U1.7 (VIOUT)
- new net: J4.1 (Pin_1), U1.1 (IP+), U1.2 (IP+)
- new net: C5.1, U1.6 (FILTER)
- new net AUX_M2: J18.2 (Pin_2)
- new net AUX_M3: J22.2 (Pin_2)
- new net AUX_M4: J23.2 (Pin_2)
- new net CSENSE: R2.2, R4.1
- new net SDA0: J24.2 (Pin_2), R5.2
- new net SDL0: J24.3 (Pin_3), R6.2
- new net VSENSE: R1.2, R3.1
Other:
- note added: "Misc. Peripheral Power"
- note added: "Power In from DC-DC converters"
- note added: "Power Out to DC-DC Converters"
- note added: "Servo Motor Capactors"
- moved on the sheet: J22, J23, J24, J28, J30, J33, JP1, Q1, Q2, R10, R11, R12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
