File: pcbs/kicad/zuko-teensy-motor-controller/_autosave-zuko-teensy-motor-controller.kicad_pcb (KiCad board)
At the start: 2 copper layers, 100 x 45 mm, 63 parts, among them J1 Conn_01x03, J10 Conn_01x03, J11 Conn_01x03, J12 Conn_01x03, J13 Conn_01x03, J14 Conn_01x02, J15 Conn_01x02, J16 Conn_01x02, J17 Conn_01x03, J18 Conn_01x03, J19 Conn_01x02, J2 Conn_01x03, J20 Conn_01x02, J21 Conn_01x02, J22 Conn_01x03, J23 Conn_01x03, J24 Conn_01x04, J25 Conn_01x03, J26 Conn_01x03, J27 Conn_01x04, J28 Conn_01x04, J29 Conn_01x04, J3 Conn_01x03, J30 Conn_01x04, J31 Conn_01x04, J32 Conn_01x04, J33 Conn_01x04, J4 Conn_01x02, J5 Conn_01x03, J6 Conn_01x03, J7 Conn_01x03, J8 Conn_01x03, J9 Conn_01x03, Q1 BSS138, Q2 BSS138, U1 ACS712xLCTR-20A, U2 Teensy4.0, U3 ULN2003

Commit message: pcb progress
Parts:
- moved R12 8.36 mm to (131.6, 59.3), turned to -90 degrees
- moved R14 6.90 mm to (121.4, 59.2), turned to -90 degrees
- moved Q2 3.05 mm to (124.7, 59.2)
- moved Q1 2.68 mm to (128.4, 59.2)
- moved J33 2.14 mm to (122.9, 54.7)
- moved J30 1.28 mm to (156.8, 69.2)
- moved J24 0.52 mm to (137.2, 54.9)
Connections:
- U2 pad 14: unconnected-(U2-Pad14) -> AUX_M1
- U2 pad 29: unconnected-(U2-Pad29) -> CSENSE
- U2 pad 30: unconnected-(U2-Pad30) -> VSENSE
- U2 pad 37: unconnected-(U2-Pad37) -> NEO2
- U2 pad 38: unconnected-(U2-Pad38) -> NEO1
- U2 pad 39: unconnected-(U2-Pad39) -> AUX_M4
- U2 pad 40: unconnected-(U2-Pad40) -> AUX_M3
- U2 pad 44: unconnected-(U2-Pad44) -> AUX_M2
