File: pcbs/kicad/zuko-teensy-motor-controller/_autosave-zuko-teensy-motor-controller.kicad_pcb (KiCad board)
At the start: 4 copper layers, 100 x 40 mm, 66 parts, among them J1 Conn_01x03, J10 Conn_01x03, J11 Conn_01x03, J12 Conn_01x03, J13 Conn_01x03, J14 Conn_01x02, J15 Conn_01x02, J16 Conn_01x02, J17 Conn_01x03, J18 Conn_01x03, J19 Conn_01x02, J2 Conn_01x03, J20 Conn_01x02, J21 Conn_01x02, J22 Conn_01x03, J23 Conn_01x02, J24 Conn_01x04, J25 Conn_01x03, J26 Conn_01x03, J27 Conn_01x04, J28 Conn_01x04, J29 Conn_01x04, J3 Conn_01x03, J30 Conn_01x04, J31 Conn_01x04, J32 Conn_01x04, J33 Conn_01x04, J34 Conn_01x02, J4 Conn_01x02, J5 Conn_01x03, J6 Conn_01x03, J7 Conn_01x03, J8 Conn_01x03, J9 Conn_01x03, Q1 BSS138, Q2 BSS138, U1 ACS712xLCTR-20A, U2 Teensy4.0, U3 ULN2003

Commit message: update notes
Parts:
- moved J4 5.32 mm to (78.7, 46.3), turned to 180 degrees
Connections:
- J4 pad 1: Net-(J4-Pad1) -> GND
- J4 pad 2: GND -> Net-(J4-Pad2)
- U1 pad 1: Net-(J4-Pad1) -> Net-(J4-Pad2)
- U1 pad 2: Net-(J4-Pad1) -> Net-(J4-Pad2)
Routing:
- net Net-(J4-Pad1): track 55.7 -> 0.00 mm, vias 2 -> 0
- net Net-(J4-Pad2): track 0.00 -> 55.6 mm, vias 0 -> 2
