File: pcbs/motor-controller/motor-controller.kicad_pcb (KiCad board)
At the start: 4 copper layers, 100 x 40 mm, 66 parts, among them J1 Conn_01x03, J10 Conn_01x03, J11 Conn_01x03, J12 Conn_01x03, J13 Conn_01x03, J14 Conn_01x02, J15 Conn_01x02, J16 Conn_01x02, J17 Conn_01x03, J18 Conn_01x03, J19 Conn_01x02, J2 Conn_01x03, J20 Conn_01x02, J21 Conn_01x02, J22 Conn_01x03, J23 Conn_01x02, J24 Conn_01x04, J25 Conn_01x03, J26 Conn_01x03, J27 Conn_01x04, J28 Conn_01x04, J29 Conn_01x04, J3 Conn_01x03, J30 Conn_01x04, J31 Conn_01x04, J32 Conn_01x04, J33 Conn_01x04, J34 Conn_01x02, J4 Conn_01x02, J5 Conn_01x03, J6 Conn_01x03, J7 Conn_01x03, J8 Conn_01x03, J9 Conn_01x03, Q1 BSS138, Q2 BSS138, U1 ACS712xLCTR-20A, U2 Teensy4.0, U3 ULN2003

Commit message: pcb update
Parts:
- added J14: Conn_01x06, Connector_PinHeader_2.54mm:PinHeader_1x06_P2.54mm_Vertical, F.Cu at (160.4, 50.2)
- renumbered C5 to C1, C6 to C2, C1 to C3, C2 to C4, C3 to C5, C4 to C6, J28 to J1, J24 to J10, J16 to J11, J19 to J12, J34 to J13, J27 to J15, J29 to J16, J31 to J17, J32 to J18, J17 to J19, J30 to J2, J1 to J20, J5 to J21, J8 to J22, J11 to J23, J25 to J24, J2 to J25, J6 to J26, J9 to J27, J12 to J28, J18 to J29, J14 to J3, J26 to J30, J3 to J31, J7 to J32, J10 to J33, J13 to J34, J22 to J35, J20 to J4, J33 to J5, J4 to J6, J15 to J7, J21 to J8, J23 to J9, JP2 to JP1, JP1 to JP2, R9 to R1, R6 to R10, R1 to R11, R3 to R12, R7 to R13, R8 to R14, R11 to R2, R10 to R3, R12 to R4, R13 to R5, R14 to R6, R2 to R7, R5 to R8, R4 to R9
Connections:
- U2 pad 2: M1 -> SPI_CS
- U2 pad 21: OUT4 -> M1
- U2 pad 22: OUT3 -> M2
- U2 pad 23: OUT2 -> NEO1
- U2 pad 24: OUT1 -> NEO2
- U2 pad 3: M2 -> SPI_MISO
- U2 pad 37: NEO2 -> SPI_MOSI
- U2 pad 38: NEO1 -> SPI_CLK
- U3 pad 1: OUT1 -> SPI_MISO
- U3 pad 2: OUT2 -> SPI_CS
- U3 pad 3: OUT3 -> SPI_CLK
- U3 pad 4: OUT4 -> SPI_MOSI
Routing:
- net SPI_MISO: track 0.00 -> 81.3 mm, vias 0 -> 2
- net SPI_CS: track 0.00 -> 77.0 mm, vias 0 -> 3
- net SPI_MOSI: track 0.00 -> 51.3 mm, vias 0 -> 2
- net SPI_CLK: track 0.00 -> 47.3 mm, vias 0 -> 2
- net M1: track 29.6 -> 68.6 mm, vias 2 -> 1
- net M2: track 30.3 -> 62.9 mm, vias 2 -> 1
- net OUT2: track 20.4 -> 0.00 mm, vias 1 -> 0
- net OUT1: track 20.2 -> 0.00 mm
- net OUT3: track 17.8 -> 0.00 mm, vias 1 -> 0
- net OUT4: track 16.9 -> 0.00 mm, vias 1 -> 0
- net +3V3: track 133.5 -> 142.7 mm
- net NEO2: track 25.8 -> 31.7 mm, vias 0 -> 1
- net NEO1: track 29.6 -> 32.8 mm
- net AUX_M3: track 42.7 -> 41.2 mm
- net Net-(J24-Pad2): track 12.4 -> 12.5 mm, vias 0 -> 1
Other:
- board text added: "HONEY BEES ATE MY PET RAPTOR!"
- board text added: "SPI"
