File: pcbs/motor-controller/motor-controller.kicad_sch (KiCad schematic)
At the start: 62 parts, among them J1 Conn_01x03, J10 Conn_01x03, J11 Conn_01x03, J12 Conn_01x03, J13 Conn_01x03, J14 Conn_01x02, J15 Conn_01x02, J16 Conn_01x02, J17 Conn_01x03, J18 Conn_01x03, J19 Conn_01x02, J2 Conn_01x03, J20 Conn_01x02, J21 Conn_01x02, J22 Conn_01x03, J23 Conn_01x02, J24 Conn_01x04, J25 Conn_01x03, J26 Conn_01x03, J27 Conn_01x04, J28 Conn_01x04, J29 Conn_01x04, J3 Conn_01x03, J30 Conn_01x04, J31 Conn_01x04, J32 Conn_01x04, J33 Conn_01x04, J34 Conn_01x02, J4 Conn_01x02, J5 Conn_01x03, J6 Conn_01x03, J7 Conn_01x03, J8 Conn_01x03, J9 Conn_01x03, Q1 BSS138, Q2 BSS138, U1 ACS712xLCTR-20A, U2 Teensy4.0, U3 ULN2003

Commit message: pcb update
Parts:
- added J14: Conn_01x06, Connector_PinHeader_2.54mm:PinHeader_1x06_P2.54mm_Vertical, symbol Connector_Generic:Conn_01x06
- renumbered C5 to C1, C6 to C2, C1 to C3, C2 to C4, C3 to C5, C4 to C6, J28 to J1, J24 to J10, J16 to J11, J19 to J12, J34 to J13, J27 to J15, J29 to J16, J31 to J17, J32 to J18, J17 to J19, J30 to J2, J1 to J20, J5 to J21, J8 to J22, J11 to J23, J25 to J24, J2 to J25, J6 to J26, J9 to J27, J12 to J28, J18 to J29, J14 to J3, J26 to J30, J3 to J31, J7 to J32, J10 to J33, J13 to J34, J22 to J35, J20 to J4, J33 to J5, J4 to J6, J15 to J7, J21 to J8, J23 to J9, JP2 to JP1, JP1 to JP2, R9 to R1, R6 to R10, R1 to R11, R3 to R12, R7 to R13, R8 to R14, R11 to R2, R10 to R3, R12 to R4, R13 to R5, R14 to R6, R2 to R7, R5 to R8, R4 to R9
Connections:
- net +3V3: now also J14.1 (Pin_1)
- net GND: now also J14.6 (Pin_6)
- net M1: now also U2.21 (14_A0_TX3_SPDIF_OUT); no longer U2.2 (0_RX1_CRX2_CS1)
- net M2: now also U2.22 (15_A1_RX3_SPDIF_IN); no longer U2.3 (1_TX1_CTX2_MISO1)
- net NEO1: now also U2.23 (16_A2_RX4_SCL1); no longer U2.38 (27_A13_SCK1)
- net NEO2: now also U2.24 (17_A3_TX4_SDA1); no longer U2.37 (26_A12_MOSI1)
- net OUT1: now also U2.3 (1_TX1_CTX2_MISO1), J14.2 (Pin_2); no longer U2.24 (17_A3_TX4_SDA1)
- net OUT2: now also U2.2 (0_RX1_CRX2_CS1), J14.5 (Pin_5); no longer U2.23 (16_A2_RX4_SCL1)
- net OUT3: now also U2.38 (27_A13_SCK1), J14.4 (Pin_4); no longer U2.22 (15_A1_RX3_SPDIF_IN)
- net OUT4: now also U2.37 (26_A12_MOSI1), J14.3 (Pin_3); no longer U2.21 (14_A0_TX3_SPDIF_OUT)
Other:
- note added: "SPI Iinterface"
- moved on the sheet: J1, J10, J11, J12, J13, J15, J16, J17, J18, J2, J3, J4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
