File: pcbs/expansion-board/expansion-board.kicad_pcb (KiCad board)
At the start: 4 copper layers, 100 x 48.5 mm, 81 parts, among them J1 Conn_01x04, J10 Conn_01x02, J12 Conn_01x06, J14 Raspberry_Pi_2_3, J15 Conn_02x03_Counter_Clockwise, J16 Conn_01x04, J17 Conn_01x04, J18 Conn_01x04, J19 Conn_01x04, J2 Conn_01x02, J20 Conn_01x03, J3 Conn_01x02, J4 Conn_01x02, J5 Conn_01x02, J6 Conn_01x02, J7 Conn_01x02, J8 Conn_01x04, J9 Conn_01x02, Q1 BSS138, U1 ACS712xLCTR-20A, U10 Conn_03x03, U2 PCA9635, U3 ADS1115IDGS, U4 ULN2003, U5 ADS1115IDGS, U6 Conn_03x03, U7 Conn_03x03, U8 Conn_03x03, U9 Conn_03x03

Commit message: expansion-board update
Parts:
- removed the J10 at (66.6, 55.1)
- removed the J2 at (66.6, 57.8)
- removed the J5 at (66.6, 67.0)
- removed the J6 at (66.6, 64.2)
- removed the J7 at (66.6, 61.5)
- removed the J9 at (66.6, 52.4)
- added J15: Conn_02x03_Odd_Even, Connector_PinHeader_2.54mm:PinHeader_2x03_P2.54mm_Vertical, F.Cu at (143.6, 44.6)
- added J3: Conn_02x03_Odd_Even, Connector_PinHeader_2.54mm:PinHeader_2x03_P2.54mm_Vertical, F.Cu at (69.1, 57.5)
- added J4: Conn_02x03_Odd_Even, Connector_PinHeader_2.54mm:PinHeader_2x03_P2.54mm_Vertical, F.Cu at (69.0, 66.3)
- JP13, JP14, JP15: moved to B.Cu
- moved U4 15.0 mm to (141.5, 55.4)
- moved R26 11.0 mm to (120.0, 57.2)
- moved R23 10.6 mm to (134.6, 52.9)
- moved R22 10.2 mm to (131.8, 52.9)
- moved JP13 9.95 mm to (85.5, 48.0), turned to 180 degrees
- moved JP15 9.93 mm to (85.5, 50.7), turned to 180 degrees
- moved JP14 9.90 mm to (85.5, 53.4), turned to 180 degrees
- moved R21 9.77 mm to (129.0, 52.9)
- moved J10 8.56 mm to (131.1, 47.0)
- moved J16 8.42 mm to (122.2, 44.5)
- moved J1 8.26 mm to (110.8, 44.5)
- moved J7 8.06 mm to (94.3, 44.5)
- moved J5 7.79 mm to (83.0, 44.5)
- moved R24 7.77 mm to (119.8, 60.9)
- moved R25 7.77 mm to (125.0, 60.9)
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- renumbered J15 to J10, J16 to J11, J17 to J12, J18 to J13, J19 to J14, J20 to J16, J4 to J2, J8 to J5, J3 to J6, J12 to J7, J14 to J9
Connections:
- J9 pad 13: unconnected-(J14-Pad13) -> GPIO27
- J9 pad 37: unconnected-(J14-Pad37) -> GPIO26
Other:
- board text added: "COMMON"
- board text added: "GPIO"
- board text removed: "COM."
- board text removed: "NEO1"

Commit message: expansion board update
Parts:
- removed JP7: SolderJumper_2_Open, Jumper:SolderJumper-2_P1.3mm_Open_Pad1.0x1.5mm
- added J1: Conn_01x02, Connector_PinHeader_2.54mm:PinHeader_1x02_P2.54mm_Vertical, F.Cu at (83.5, 44.4)
- added JP10: Jumper_2_Open, Jumper:SolderJumper-2_P1.3mm_Open_Pad1.0x1.5mm, F.Cu at (154.1, 66.1)
- added JP11: Jumper_2_Open, Jumper:SolderJumper-2_P1.3mm_Open_Pad1.0x1.5mm, F.Cu at (151.3, 66.1)
- added JP12: Jumper_2_Open, Jumper:SolderJumper-2_P1.3mm_Open_Pad1.0x1.5mm, F.Cu at (148.6, 66.1)
- added JP9: Jumper_2_Open, Jumper:SolderJumper-2_P1.3mm_Open_Pad1.0x1.5mm, F.Cu at (156.9, 66.1)
- added R27: 3.9k, Resistor_SMD:R_1206_3216Metric_Pad1.30x1.75mm_HandSolder, F.Cu at (99.1, 52.1)
- added R28: 3.9k, Resistor_SMD:R_1206_3216Metric_Pad1.30x1.75mm_HandSolder, F.Cu at (99.1, 49.5)
- added U7: 24LC256, Package_SO:SOIC-8_3.9x4.9mm_P1.27mm, F.Cu at (92.5, 50.8)
- H3, H4, H5, H6: footprint MountingHole:MountingHole_2.5mm -> General:RPi_Hat_Mounting_Hole
- JP13, JP14, JP15: moved to F.Cu
- moved JP13 11.9 mm to (74.6, 53.0), turned to 90 degrees
- moved JP14 8.46 mm to (77.1, 53.0), turned to 90 degrees
- moved J9 7.33 mm to (138.4, 47.0)
- moved J6 7.13 mm to (129.3, 44.4)
- moved J14 7.03 mm to (117.8, 44.4)
- moved J16 6.91 mm to (101.2, 44.4)
- moved J15 6.80 mm to (89.8, 44.4)
- moved JP15 6.38 mm to (79.6, 53.0), turned to 90 degrees
- moved J7 6.24 mm to (149.9, 44.4)
- moved C1 4.31 mm to (90.3, 61.8)
- moved JP1 3.84 mm to (92.7, 56.0)
- moved JP2 3.56 mm to (95.0, 56.0)
- moved R22 3.53 mm to (125.8, 51.2)
- moved R23 3.53 mm to (128.7, 51.2)
- moved R24 3.53 mm to (131.4, 51.2)
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- renumbered C4 to C1, C1 to C2, C2 to C3, C8 to C4, C3 to C5, C5 to C6, C6 to C7, C7 to C8, J11 to J10, J12 to J11, J13 to J12, J14 to J13, J1 to J14, J5 to J15, J7 to J16, J6 to J5, J16 to J6, J15 to J7, J9 to J8, J10 to J9, R5 to R1, R17 to R10, R12 to R11, R13 to R12, R14 to R13, R24 to R14, R25 to R15, R15 to R16, R16 to R17, R26 to R19, R19 to R20, R20 to R21, R21 to R22, R22 to R23, R23 to R24, R1 to R25, R3 to R26, R4 to R3, R8 to R4, R6 to R5, R7 to R6, R9 to R7, R10 to R8, R11 to R9, U3 to U1, U9 to U11, U1 to U2, U2 to U3, U5 to U4, U4 to U5, U7 to U8, U8 to U9
Connections:
- J8 pad 27: unconnected-(J9-Pad27) -> ID_SD
- J8 pad 28: unconnected-(J9-Pad28) -> ID_SC
Other:
- board size 100 x 48.5 mm -> 100 x 49.8 mm
- board text added: "ADC"
- board text added: "ADC1"
- board text added: "ADC2"
- board text added: "AUX SERVO"
- board text added: "CLK"
- board text added: "CS"
- board text added: "MISO"
- board text added: "MOSI"
- board text added: "PIN"
- board text added: "RX"
- board text added: "SEN"
- board text added: "SIG"
- board text added: "TX"
- board text removed: "3V3"
- board text removed: "A1"
- board text removed: "A2"
- board text removed: "A3"
- board text removed: "AUX SRV."
- board text removed: "COMMON"
- board text removed: "Rx"
- board text removed: "SW"
- board text removed: "Tx"

Commit message: expansion board update
Parts:
- removed the R25 at (116.5, 52.8)
- removed the R26 at (121.5, 52.8)
- added C3: 10uF, Capacitor_SMD:C_0805_2012Metric, F.Cu at (104.8, 64.4)
- added R10: 1.2k, Resistor_SMD:R_0805_2012Metric, F.Cu at (130.0, 58.0)
- added R12: 1.2k, Resistor_SMD:R_0805_2012Metric, F.Cu at (128.9, 66.0)
- C1, C2: footprint Capacitor_SMD:C_1206_3216Metric_Pad1.33x1.80mm_HandSolder -> Capacitor_SMD:C_0805_2012Metric
- C4: renamed from C3; footprint Capacitor_SMD:C_1206_3216Metric_Pad1.33x1.80mm_HandSolder -> Capacitor_SMD:C_0805_2012Metric
- C5: renamed from C4; footprint Capacitor_SMD:C_1206_3216Metric_Pad1.33x1.80mm_HandSolder -> Capacitor_SMD:C_0805_2012Metric
- R1: renamed from R3; footprint Resistor_SMD:R_1206_3216Metric_Pad1.30x1.75mm_HandSolder -> Resistor_SMD:R_0805_2012Metric
- R11: renamed from R2; footprint Resistor_SMD:R_1206_3216Metric_Pad1.30x1.75mm_HandSolder -> Resistor_SMD:R_0805_2012Metric
- R13: renamed from R11; footprint Resistor_SMD:R_1206_3216Metric_Pad1.30x1.75mm_HandSolder -> Resistor_SMD:R_0805_2012Metric
- R14: renamed from R12; footprint Resistor_SMD:R_1206_3216Metric_Pad1.30x1.75mm_HandSolder -> Resistor_SMD:R_0805_2012Metric
- R15: renamed from R13; footprint Resistor_SMD:R_1206_3216Metric_Pad1.30x1.75mm_HandSolder -> Resistor_SMD:R_0805_2012Metric
- R16: renamed from R14; footprint Resistor_SMD:R_1206_3216Metric_Pad1.30x1.75mm_HandSolder -> Resistor_SMD:R_0805_2012Metric
- R17: renamed from R15; footprint Resistor_SMD:R_1206_3216Metric_Pad1.30x1.75mm_HandSolder -> Resistor_SMD:R_0805_2012Metric
- R18: renamed from R16; footprint Resistor_SMD:R_1206_3216Metric_Pad1.30x1.75mm_HandSolder -> Resistor_SMD:R_0805_2012Metric
- R19: renamed from R17; footprint Resistor_SMD:R_1206_3216Metric_Pad1.30x1.75mm_HandSolder -> Resistor_SMD:R_0805_2012Metric
- R2: renamed from R1; footprint Resistor_SMD:R_1206_3216Metric_Pad1.30x1.75mm_HandSolder -> Resistor_SMD:R_0805_2012Metric
- R20: renamed from R18; footprint Resistor_SMD:R_1206_3216Metric_Pad1.30x1.75mm_HandSolder -> Resistor_SMD:R_0805_2012Metric
- R21: renamed from R19; footprint Resistor_SMD:R_1206_3216Metric_Pad1.30x1.75mm_HandSolder -> Resistor_SMD:R_0805_2012Metric
- R22: renamed from R20; footprint Resistor_SMD:R_1206_3216Metric_Pad1.30x1.75mm_HandSolder -> Resistor_SMD:R_0805_2012Metric
- R23: renamed from R21; footprint Resistor_SMD:R_1206_3216Metric_Pad1.30x1.75mm_HandSolder -> Resistor_SMD:R_0805_2012Metric
- R24: renamed from R22; footprint Resistor_SMD:R_1206_3216Metric_Pad1.30x1.75mm_HandSolder -> Resistor_SMD:R_0805_2012Metric
- R25: renamed from R23; footprint Resistor_SMD:R_1206_3216Metric_Pad1.30x1.75mm_HandSolder -> Resistor_SMD:R_0805_2012Metric
- R26: renamed from R24; footprint Resistor_SMD:R_1206_3216Metric_Pad1.30x1.75mm_HandSolder -> Resistor_SMD:R_0805_2012Metric
- R27, R28: footprint Resistor_SMD:R_1206_3216Metric_Pad1.30x1.75mm_HandSolder -> Resistor_SMD:R_0805_2012Metric
- R3: renamed from R5; footprint Resistor_SMD:R_1206_3216Metric_Pad1.30x1.75mm_HandSolder -> Resistor_SMD:R_0805_2012Metric
- R4: renamed from R6; footprint Resistor_SMD:R_1206_3216Metric_Pad1.30x1.75mm_HandSolder -> Resistor_SMD:R_0805_2012Metric
- R5: renamed from R4; footprint Resistor_SMD:R_1206_3216Metric_Pad1.30x1.75mm_HandSolder -> Resistor_SMD:R_0805_2012Metric
- R6: renamed from R7; footprint Resistor_SMD:R_1206_3216Metric_Pad1.30x1.75mm_HandSolder -> Resistor_SMD:R_0805_2012Metric
- R7: renamed from R8; footprint Resistor_SMD:R_1206_3216Metric_Pad1.30x1.75mm_HandSolder -> Resistor_SMD:R_0805_2012Metric
- R8: renamed from R9; footprint Resistor_SMD:R_1206_3216Metric_Pad1.30x1.75mm_HandSolder -> Resistor_SMD:R_0805_2012Metric
- R9: renamed from R10; footprint Resistor_SMD:R_1206_3216Metric_Pad1.30x1.75mm_HandSolder -> Resistor_SMD:R_0805_2012Metric
- moved JP7 21.2 mm to (123.2, 52.8), turned to -90 degrees
- moved JP1 12.1 mm to (104.8, 55.5)
- moved JP6 11.8 mm to (92.0, 55.5)
- moved JP2 7.32 mm to (102.3, 55.5)
- moved R13 7.26 mm to (91.8, 63.9)
- moved JP5 7.02 mm to (94.5, 55.5)
- moved R20 5.20 mm to (131.8, 64.4), turned to 90 degrees
- moved C1 5.06 mm to (91.5, 66.7)
- moved R17 4.13 mm to (127.0, 58.0), turned to 90 degrees
- moved JP3 2.58 mm to (99.7, 55.5)
- moved J5 2.55 mm to (69.0, 49.0), turned to -90 degrees
- moved JP4 2.29 mm to (97.1, 55.5)
- moved R19 2.05 mm to (79.4, 60.8)
- moved C5 1.90 mm to (137.4, 67.2)
- moved JP14 1.90 mm to (80.4, 54.7)
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- renumbered C5 to C6, C6 to C7, C7 to C8, C8 to C9, JP11 to JP10, JP12 to JP11, JP13 to JP12, JP14 to JP13, JP15 to JP14, JP8 to JP7, JP9 to JP8, JP10 to JP9
Connections:
- J14 pad 2: SDA5 -> SDAXXX
- J14 pad 3: SCL5 -> SCLXXX
- MOD1 pad 4: SDA1 -> SDA5
- MOD1 pad 5: SCL1 -> SCL5
- R2 pad 2: SDA1 -> SDA5
- R5 pad 2: SCL1 -> SCL5
- U1 pad 4: CSENSE -> VSENSE
- U1 pad 5: VSENSE -> CSENSE
- U3 pad 10: M5 -> unconnected-(U3-Pad10)
- U3 pad 11: M6 -> AUX_M3
- U3 pad 12: M7 -> AUX_M2
- U3 pad 13: M8 -> AUX_M1
- U3 pad 15: M9 -> M1
- U3 pad 16: M10 -> M2
- U3 pad 17: M11 -> M3
- U3 pad 18: M12 -> M4
- U3 pad 19: AUX_M1 -> M5
- U3 pad 20: AUX_M2 -> M6
- U3 pad 21: AUX_M3 -> M7
- U3 pad 22: unconnected-(U3-Pad22) -> M8
- U3 pad 6: M1 -> M12
- U3 pad 7: M2 -> M11
- U3 pad 8: M3 -> M10
- U3 pad 9: M4 -> M9
Routing:
- net +3V3: track 0.00 -> 347.9 mm, vias 0 -> 9
- net SCL6: track 0.00 -> 96.1 mm
- net SDA6: track 0.00 -> 90.9 mm
- net GND: track 0.00 -> 89.9 mm, vias 0 -> 19
- net SDA1: track 0.00 -> 85.7 mm, vias 0 -> 3
- net SCL1: track 0.00 -> 80.2 mm, vias 0 -> 3
- net OUT3: track 0.00 -> 72.3 mm, vias 0 -> 2
- net Net-(J8-Pad29): track 0.00 -> 71.2 mm, vias 0 -> 3
- net OUT4: track 0.00 -> 69.0 mm, vias 0 -> 3
- net Net-(J8-Pad31): track 0.00 -> 66.3 mm, vias 0 -> 2
- net OUT5: track 0.00 -> 62.9 mm, vias 0 -> 2
- net TX: track 0.00 -> 61.1 mm, vias 0 -> 2
- net Net-(J8-Pad26): track 0.00 -> 59.0 mm, vias 0 -> 4
- net M11: track 0.00 -> 58.1 mm, vias 0 -> 3
- net OUT1: track 0.00 -> 55.6 mm, vias 0 -> 3
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- added copper zone on B.Cu, net +BATT
- added copper zone on F.Cu, net +BATT
- added copper zone on In1.Cu, net +BATT
- added copper zone on In2.Cu, net +BATT
- added copper zone on B.Cu, net GND
- added copper zone on F.Cu, net GND
- added copper zone on In1.Cu, net GND
- added copper zone on In2.Cu, net GND
Other:
- board text added: "+A"
- board text added: "+B"
- board text added: "A0"
- board text added: "A1"
- board text added: "A2"
- board text added: "A3"
- board text added: "A4"
- board text added: "A5"
- board text added: "C"
- board text added: "ZUKO - A ROBOT DOG! Expansion Board v1"
- board text removed: "+AUX"
- board text removed: "+BATT"
- board text removed: "SIG."
- board text removed: "ZUKO - A ROBOT DOG! MOTOR CTRL. - 2022 - V2"

Commit message: expansion board update
Parts:
- removed the J7 at (149.9, 44.4)
- removed JP11, JP8: Jumper_2_Open, Jumper:SolderJumper-2_P1.3mm_Open_Pad1.0x1.5mm
- removed the JP2 at (102.3, 55.5)
- removed the JP3 at (99.7, 55.5)
- removed the JP5 at (94.5, 55.5)
- removed the JP6 at (92.0, 55.5)
- removed the JP7 at (123.2, 52.8)
- removed the R1 at (108.8, 62.3)
- removed the R11 at (108.8, 64.7)
- removed the R13 at (91.8, 63.9)
- removed R20: 10k, Resistor_SMD:R_0805_2012Metric
- removed R24, R25, R26: 500Ω, Resistor_SMD:R_0805_2012Metric
- removed the R3 at (108.8, 59.9)
- removed the R4 at (108.8, 57.4)
- removed the R7 at (108.8, 52.6)
- removed the R8 at (108.8, 50.1)
- removed the R9 at (85.1, 63.9)
- added C10: C_Polarized, Capacitor_SMD:CP_Elec_10x10, F.Cu at (148.9, 44.5)
- added D1: D_Schottky, Diode_SMD:D_SMC, F.Cu at (158.2, 52.2)
- added L1: L, Inductor_SMD:L_12x12mm_H6mm, F.Cu at (136.5, 62.1)
- added R18: 3.9k, Resistor_SMD:R_0805_2012Metric, F.Cu at (160.0, 70.2)
- added R19: 1.21k, Resistor_SMD:R_0805_2012Metric, F.Cu at (160.0, 72.3)
- added R5: 1.2k, Resistor_SMD:R_0805_2012Metric, F.Cu at (90.2, 65.8)
- added U12: LM2596S-5, Package_TO_SOT_SMD:TO-263-5_TabPin3, F.Cu at (153.3, 63.2)
- JP1, JP4: value SolderJumper_2_Open -> Jumper_2_Open; moved to B.Cu
- JP2: renamed from JP9; moved to B.Cu
- JP3: renamed from JP10; moved to B.Cu
- JP5: renamed from JP12; moved to B.Cu
- JP6: renamed from JP13; moved to B.Cu
- JP7: renamed from JP14; moved to B.Cu
- R6: value 10k -> 1.2k
- moved J3 81.8 mm to (150.6, 51.9), turned to -90 degrees
- moved JP2 70.2 mm to (85.0, 55.5)
- moved J11 67.2 mm to (87.9, 44.1)
- moved J9 67.2 mm to (82.3, 44.1)
- moved J10 67.2 mm to (85.1, 44.1)
- moved J12 67.2 mm to (90.7, 44.1)
- moved JP3 64.1 mm to (88.0, 55.5)
- moved R15 52.1 mm to (90.2, 61.8)
- moved R14 52.1 mm to (90.2, 59.6)
- moved U4 51.1 mm to (85.2, 60.8)
- moved C5 50.3 mm to (87.2, 63.7)
- moved J7 43.2 mm to (95.2, 46.7)
- moved J14 42.9 mm to (132.8, 44.1)
- moved U5 41.1 mm to (98.5, 55.6), turned to 180 degrees
- moved JP1 22.9 mm to (81.9, 55.5), turned to 90 degrees
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- renumbered C3 to C1, C1 to C2, C2 to C3, J11 to J10, J12 to J11, J13 to J12, J14 to J13, J15 to J14, J16 to J15, J9 to J7, J10 to J9, R10 to R1, R17 to R10, R18 to R11, R19 to R12, R21 to R13, R22 to R14, R23 to R15, R27 to R16, R28 to R17, R12 to R2, R2 to R3, R5 to R4, R14 to R7, R15 to R8, R16 to R9, U3 to U2, U2 to U3
Connections:
- net Net-(J2-Pad2) renamed /+BATT-RAW
- J13 pad 2: SDAXXX -> SDA5
- J13 pad 3: SCLXXX -> SCL5
- J15 pad 2: SPI_MISO -> SPI_CLK
- J15 pad 4: SPI_CLK -> SPI_MISO
- J7 pad 1: Net-(J9-Pad1) -> Net-(J7-Pad1)
- J7 pad 2: Net-(J9-Pad2) (its old number) -> +3V3
- J7 pad 4: Net-(J9-Pad4) -> +3V3
- J7 pad 5: Net-(J9-Pad5) -> Net-(J7-Pad5)
- J7 pad 6: Net-(J9-Pad6) -> +3V3
- J8 pad 11: OUT2 -> OUT3
- J8 pad 12: NEOPIXEL -> SPI_CS
- J8 pad 13: GPIO27 -> OUT4
- J8 pad 18: OUT6 -> OUT5
- J8 pad 19: SPI_MOSI -> NEOPIXEL
- J8 pad 21: SPI_MISO -> OUT7
- J8 pad 22: OUT7 -> OUT6
- J8 pad 23: SPI_CLK -> Net-(J8-Pad23)
- J8 pad 24: SPI_CS -> SDA4
- J8 pad 26: Net-(J8-Pad26) -> SCL4
- J8 pad 35: OUT3 -> SPI_MISO
- J8 pad 37: GPIO26 -> Net-(J8-Pad37)
- J8 pad 38: OUT4 -> SPI_MOSI
- J8 pad 40: OUT5 -> SPI_CLK
- J8 pad 7: Net-(J8-Pad7) -> OUT2
- JP1 pad 1: +3V3 -> Net-(J8-Pad37)
- JP1 pad 2: Net-(JP1-Pad2) -> FOOT1
- JP2 pad 2: FOOT3 -> FOOT2
- JP3 pad 2: FOOT2 -> FOOT3
- JP4 pad 1: +3V3 -> Net-(J8-Pad23)
- JP4 pad 2: Net-(JP4-Pad2) -> FOOT4
- MOD1 pad 7: Net-(JP7-Pad1) -> unconnected-(MOD1-Pad7)
- R14 pad 2: SDA6 -> SDA4
- R15 pad 2: SCL6 -> SCL4
- R6 pad 1: Net-(JP3-Pad2) -> +3V3
- R6 pad 2: GND -> SCL6
- U1 pad 1: Net-(R9-Pad1) -> GND
- U2 pad 1: Net-(JP1-Pad2) -> GND
- U2 pad 2: Net-(JP2-Pad2) -> GND
- U2 pad 23: Net-(R13-Pad1) -> GND
- U2 pad 24: Net-(JP6-Pad2) (its old number) -> GND
- U2 pad 25: Net-(R11-Pad1) -> GND
- U2 pad 3: Net-(JP3-Pad2) -> GND
- U2 pad 4: Net-(JP4-Pad2) -> GND
- U2 pad 5: Net-(JP5-Pad2) (its old number) -> GND
- U4 pad 1: Net-(R20-Pad2) -> GND
- U4 pad 10: SDA6 -> SDA4
- U4 pad 9: SCL6 -> SCL4
- U5 pad 10: Net-(J9-Pad5) -> Net-(J7-Pad1)
- U5 pad 12: Net-(J9-Pad1) -> Net-(J7-Pad5)
Routing:
- net +3V3: track 347.9 -> 52.7 mm, vias 9 -> 10
- net +5V: track 23.4 -> 161.3 mm, vias 0 -> 4
- net SCL4: track 0.00 -> 71.7 mm
- net SDA4: track 0.00 -> 61.6 mm
- net Net-(J8-Pad26): track 59.0 -> 0.00 mm, vias 4 -> 0
- net Net-(J8-Pad23): track 0.00 -> 56.5 mm, vias 0 -> 2
- net GPIO26: track 54.3 -> 0.00 mm, vias 1 -> 0
- net Net-(J8-Pad37): track 0.00 -> 51.0 mm, vias 0 -> 2
- net Net-(J8-Pad7): track 48.4 -> 0.00 mm, vias 2 -> 0
- net RX: track 53.9 -> 10.2 mm, vias 1 -> 0
- net Net-(JP6-Pad2) (its old number): track 40.6 -> 0.00 mm, vias 4 -> 0
- net TX: track 61.1 -> 22.4 mm, vias 2 -> 0
- net Net-(D1-Pad1): track 0.00 -> 36.6 mm
- net OUT2: track 36.7 -> 71.9 mm
- net Net-(JP5-Pad2) (its old number): track 30.2 -> 0.00 mm, vias 2 -> 0
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- added copper zone on In2.Cu, net +3V3
- added copper zone on B.Cu, net /+BATT-RAW
- added copper zone on F.Cu, net /+BATT-RAW
- added copper zone on In1.Cu, net /+BATT-RAW
- added copper zone on In2.Cu, net /+BATT-RAW
Other:
- board text added: "4"
- board text added: "A"
- board text added: "B"
- board text added: "F."
- board text added: "G."
- board text added: "L."
- board text removed: "+A"
- board text removed: "+B"
- board text removed: "A0"
- board text removed: "A1"
- board text removed: "A2"
- board text removed: "A3"
- board text removed: "A4"
- board text removed: "A5"
- board text removed: "ADC1"
- board text removed: "ADC2"
- board text removed: "GPIO"
- board text removed: "PIN"
- board text removed: "SEN"

Commit message: expansion board update
Parts:
- removed the R18 at (160.0, 70.2)
- added D1: LED, LED_SMD:LED_0805_2012Metric, F.Cu at (66.4, 70.6)
- added R4: 10k, Resistor_SMD:R_0805_2012Metric, F.Cu at (66.4, 72.8)
- added RV1: 50k, General:Precision_pot, F.Cu at (149.6, 53.0)
- C7: renamed from C10; value C_Polarized -> 560uF
- L1: value L -> 22uH
- moved J3 11.3 mm to (139.8, 48.7), turned to 0 degrees
- moved J6 2.63 mm to (133.4, 48.7), turned to 0 degrees
- moved R17 2.32 mm to (159.8, 70.0), turned to 180 degrees
- moved C7 0.63 mm to (149.6, 44.5)
- moved L1 0.40 mm to (136.5, 62.5)
- moved D2 0.19 mm to (158.4, 52.2)
- renumbered C9 to C10, C7 to C8, C8 to C9, D1 to D2, J11 to J10, J12 to J11, J8 to J12, J9 to J8, J10 to J9, R8 to R10, R10 to R11, R11 to R12, R12 to R13, R13 to R14, R14 to R15, R15 to R16, R19 to R17, R16 to R18, R17 to R19, R4 to R5, R5 to R6, R6 to R7, R7 to R8, U9 to U10, U10 to U12, U5 to U4, U4 to U5, U12 to U6, U6 to U8, U8 to U9
Connections:
- R17 pad 1: +5V -> GND
- R17 pad 2: GND -> Net-(R17-Pad2)
- U6 pad 4: Net-(R18-Pad1) -> Net-(R17-Pad2)
Routing:
- net Net-(R17-Pad2): track 0.00 -> 41.6 mm, vias 0 -> 2
- net Net-(D2-Pad1): track 36.6 -> 63.3 mm, vias 0 -> 6
- net +BATT: track 58.8 -> 79.2 mm, vias 3 -> 8
- net Net-(R18-Pad1): track 15.8 -> 0.00 mm, vias 2 -> 0
- net GND: track 89.7 -> 102.0 mm, vias 41 -> 40
- net /+BATT-RAW: track 0.00 -> 4.61 mm
- net Net-(J6-Pad2): track 21.5 -> 17.5 mm
- net +5V: track 161.3 -> 164.9 mm, vias 4 -> 7
- net +3V3: track 52.7 -> 56.0 mm
- net SDA1: track 56.5 -> 53.5 mm
- net Net-(D1-Pad2): track 0.00 -> 2.99 mm
- net SCL1: track 55.6 -> 54.7 mm
- net OUT3: track 58.5 -> 59.3 mm
Other:
- board text added: "I2C"
- board text removed: "I2C AUX"
