File: pcbs/expansion-board/expansion-board.kicad_pcb (KiCad board)
At the start: 4 copper layers, 100 x 49.8 mm, 75 parts, among them J1 Conn_01x02, J10 Conn_01x04, J11 Conn_01x04, J12 Raspberry_Pi_2_3, J13 Conn_01x04, J14 Conn_01x04, J15 Conn_01x06, J2 Conn_01x02, J3 Conn_02x03_Odd_Even, J4 Conn_02x03_Odd_Even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

Commit message: minor expansion board fixes
Routing:
- net +BATT: track 79.2 -> 75.3 mm
- net +5V: track 164.9 -> 164.2 mm
- net OUT3: track 59.3 -> 59.9 mm
- net OUT4: track 57.0 -> 57.6 mm
- net /+BATT-RAW: vias 2 -> 4

Commit message: expansion board v1.0 release
Parts:
- moved J3 3.93 mm to (142.7, 51.3), turned to -90 degrees
- moved D2 0.61 mm to (159.0, 52.2)
- moved RV1 0.54 mm to (150.1, 53.0)
Routing:
- net Net-(R17-Pad2): track 41.6 -> 31.8 mm
- net +3V3: track 56.0 -> 59.2 mm, vias 10 -> 11
- net +5V: track 164.2 -> 161.6 mm
Other:
- board text added: "NEO"
- board text added: "ZUKO - A ROBOT DOG! Expansion Board v1.0"
- board text removed: "NEOPIXEL"
- board text removed: "ZUKO - A ROBOT DOG! Expansion Board v1"
