File: pcbs/expansion-board/expansion-board.kicad_sch (KiCad schematic)
At the start: 86 parts, among them J1 Conn_01x04, J10 Conn_01x02, J12 Conn_01x06, J13 Conn_01x02, J14 Raspberry_Pi_2_3, J15 Conn_02x03_Counter_Clockwise, J16 Conn_01x04, J17 Conn_01x04, J18 Conn_01x04, J19 Conn_01x04, J2 Conn_01x02, J20 Conn_01x03, J3 Conn_01x02, J4 Conn_01x02, J5 Conn_01x02, J6 Conn_01x02, J7 Conn_01x02, J8 Conn_01x04, J9 Conn_01x02, Q1 BSS138, U1 ACS712xLCTR-20A, U10 Conn_03x03, U2 PCA9635, U3 ADS1115IDGS, U4 ULN2003, U5 ADS1115IDGS, U6 Conn_03x03, U7 Conn_03x03, U8 Conn_03x03, U9 Conn_03x03

Commit message: expansion-board update
Parts:
- removed J10, J2, J5, J6, J7, J9: Conn_01x02, Connector_PinHeader_2.54mm:PinHeader_1x02_P2.54mm_Vertical, symbol Connector_Generic:Conn_01x02
- added J15, J3, J4: Conn_02x03_Odd_Even, Connector_PinHeader_2.54mm:PinHeader_2x03_P2.54mm_Vertical, symbol Connector_Generic:Conn_02x03_Odd_Even
- renumbered J15 to J10, J16 to J11, J17 to J12, J18 to J13, J19 to J14, J20 to J16, J4 to J2, J8 to J5, J3 to J6, J12 to J7, J13 to J8, J14 to J9
Connections:
- net +3V3: now also J15.1 (Pin_1), J15.2 (Pin_2)
- net +5V: now also J3.1 (Pin_1), J3.3 (Pin_3), J3.5 (Pin_5)
- net +BATT: now also J4.1 (Pin_1), J4.3 (Pin_3), J4.5 (Pin_5)
- net GND: now also J15.5 (Pin_5), J15.6 (Pin_6), J3.2 (Pin_2), J3.4 (Pin_4), J3.6 (Pin_6), J4.2 (Pin_2), J4.4 (Pin_4), J4.6 (Pin_6)
- net GPIO27: now reaches J9.13 (GPIO27)
- net GPIO27: now also J15.4 (Pin_4)
- net GPIO26: now reaches J9.37 (GPIO26)
- net GPIO26: now also J15.3 (Pin_3)
- no-connect marks 9 -> 11
Other:
- note added: "Extra GPIO Breakout"
- note added: "Power Connectors To/From DC-DC Convertors"
- note removed: "Extra Power Connections"
- note removed: "Power In from DC-DC converters"
- note removed: "Power Out to DC-DC Converters"
- moved on the sheet: C1, C2, C3, C4, C5, C6, C7, C8, H1, H2, H3, H4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

Commit message: expansion board update
Parts:
- removed JP7: SolderJumper_2_Open, Jumper:SolderJumper-2_P1.3mm_Open_Pad1.0x1.5mm, symbol Jumper:SolderJumper_2_Open
- added R27, R28: 3.9k, Resistor_SMD:R_1206_3216Metric_Pad1.30x1.75mm_HandSolder, symbol Device:R_Small_US
- added U7: 24LC256, Package_SO:SOIC-8_3.9x4.9mm_P1.27mm, symbol Memory_EEPROM:24LC256
- H3, H4, H5, H6: footprint MountingHole:MountingHole_2.5mm -> General:RPi_Hat_Mounting_Hole
- J1: renamed from J8; footprint (none) -> Connector_PinHeader_2.54mm:PinHeader_1x02_P2.54mm_Vertical
- JP10, JP11, JP12, JP9: footprint (none) -> Jumper:SolderJumper-2_P1.3mm_Open_Pad1.0x1.5mm
- renumbered C4 to C1, C1 to C2, C2 to C3, C8 to C4, C3 to C5, C5 to C6, C6 to C7, C7 to C8, J11 to J10, J12 to J11, J13 to J12, J14 to J13, J1 to J14, J5 to J15, J7 to J16, J6 to J5, J16 to J6, J15 to J7, J9 to J8, J10 to J9, R5 to R1, R17 to R10, R12 to R11, R13 to R12, R14 to R13, R24 to R14, R25 to R15, R15 to R16, R16 to R17, R26 to R19, R19 to R20, R20 to R21, R21 to R22, R22 to R23, R23 to R24, R1 to R25, R3 to R26, R4 to R3, R8 to R4, R6 to R5, R7 to R6, R9 to R7, R10 to R8, R11 to R9, U3 to U1, U9 to U11, U1 to U2, U2 to U3, U5 to U4, U4 to U5, U7 to U8, U8 to U9
Connections:
- net +3V3: now also R27.1, R28.1, U7.8 (VCC)
- net GND: now also U7.1 (A0), U7.2 (A1), U7.3 (A2), U7.4 (GND)
- net ID_SD: now reaches J8.27 (ID_SD/GPIO0)
- net ID_SD: now also R27.2, U7.5 (SDA)
- net ID_SC: now reaches J8.28 (ID_SC/GPIO1)
- net ID_SC: now also R28.2, U7.6 (SCL)
- no-connect marks 11 -> 10
Other:
- note added: "Optional ID EEPROM"
- note added: "See: https://github.com/raspberrypi/hats"
- moved on the sheet: C1, C2, C3, C4, C5, C6, C7, C8, H1, H2, H3, H4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

Commit message: expansion board update
Parts:
- removed R25, R26: 1.2k, Resistor_SMD:R_1206_3216Metric_Pad1.30x1.75mm_HandSolder, symbol Device:R_Small_US
- added C3: 10uF, Capacitor_SMD:C_0805_2012Metric, symbol Device:C
- added R10, R12: 1.2k, Resistor_SMD:R_0805_2012Metric, symbol Device:R_Small_US
- C1, C2: footprint Capacitor_SMD:C_1206_3216Metric_Pad1.33x1.80mm_HandSolder -> Capacitor_SMD:C_0805_2012Metric
- C4: renamed from C3; footprint Capacitor_SMD:C_1206_3216Metric_Pad1.33x1.80mm_HandSolder -> Capacitor_SMD:C_0805_2012Metric
- C5: renamed from C4; footprint Capacitor_SMD:C_1206_3216Metric_Pad1.33x1.80mm_HandSolder -> Capacitor_SMD:C_0805_2012Metric
- R1: renamed from R3; footprint Resistor_SMD:R_1206_3216Metric_Pad1.30x1.75mm_HandSolder -> Resistor_SMD:R_0805_2012Metric
- R11: renamed from R2; footprint Resistor_SMD:R_1206_3216Metric_Pad1.30x1.75mm_HandSolder -> Resistor_SMD:R_0805_2012Metric
- R13: renamed from R11; footprint Resistor_SMD:R_1206_3216Metric_Pad1.30x1.75mm_HandSolder -> Resistor_SMD:R_0805_2012Metric
- R14: renamed from R12; footprint Resistor_SMD:R_1206_3216Metric_Pad1.30x1.75mm_HandSolder -> Resistor_SMD:R_0805_2012Metric
- R15: renamed from R13; footprint Resistor_SMD:R_1206_3216Metric_Pad1.30x1.75mm_HandSolder -> Resistor_SMD:R_0805_2012Metric
- R16: renamed from R14; footprint Resistor_SMD:R_1206_3216Metric_Pad1.30x1.75mm_HandSolder -> Resistor_SMD:R_0805_2012Metric
- R17: renamed from R15; footprint Resistor_SMD:R_1206_3216Metric_Pad1.30x1.75mm_HandSolder -> Resistor_SMD:R_0805_2012Metric
- R18: renamed from R16; footprint Resistor_SMD:R_1206_3216Metric_Pad1.30x1.75mm_HandSolder -> Resistor_SMD:R_0805_2012Metric
- R19: renamed from R17; footprint Resistor_SMD:R_1206_3216Metric_Pad1.30x1.75mm_HandSolder -> Resistor_SMD:R_0805_2012Metric
- R2: renamed from R1; footprint Resistor_SMD:R_1206_3216Metric_Pad1.30x1.75mm_HandSolder -> Resistor_SMD:R_0805_2012Metric
- R20: renamed from R18; footprint Resistor_SMD:R_1206_3216Metric_Pad1.30x1.75mm_HandSolder -> Resistor_SMD:R_0805_2012Metric
- R21: renamed from R19; footprint Resistor_SMD:R_1206_3216Metric_Pad1.30x1.75mm_HandSolder -> Resistor_SMD:R_0805_2012Metric
- R22: renamed from R20; footprint Resistor_SMD:R_1206_3216Metric_Pad1.30x1.75mm_HandSolder -> Resistor_SMD:R_0805_2012Metric
- R23: renamed from R21; footprint Resistor_SMD:R_1206_3216Metric_Pad1.30x1.75mm_HandSolder -> Resistor_SMD:R_0805_2012Metric
- R24: renamed from R22; footprint Resistor_SMD:R_1206_3216Metric_Pad1.30x1.75mm_HandSolder -> Resistor_SMD:R_0805_2012Metric
- R25: renamed from R23; footprint Resistor_SMD:R_1206_3216Metric_Pad1.30x1.75mm_HandSolder -> Resistor_SMD:R_0805_2012Metric
- R26: renamed from R24; footprint Resistor_SMD:R_1206_3216Metric_Pad1.30x1.75mm_HandSolder -> Resistor_SMD:R_0805_2012Metric
- R27, R28: footprint Resistor_SMD:R_1206_3216Metric_Pad1.30x1.75mm_HandSolder -> Resistor_SMD:R_0805_2012Metric
- R3: renamed from R5; footprint Resistor_SMD:R_1206_3216Metric_Pad1.30x1.75mm_HandSolder -> Resistor_SMD:R_0805_2012Metric
- R4: renamed from R6; footprint Resistor_SMD:R_1206_3216Metric_Pad1.30x1.75mm_HandSolder -> Resistor_SMD:R_0805_2012Metric
- R5: renamed from R4; footprint Resistor_SMD:R_1206_3216Metric_Pad1.30x1.75mm_HandSolder -> Resistor_SMD:R_0805_2012Metric
- R6: renamed from R7; footprint Resistor_SMD:R_1206_3216Metric_Pad1.30x1.75mm_HandSolder -> Resistor_SMD:R_0805_2012Metric
- R7: renamed from R8; footprint Resistor_SMD:R_1206_3216Metric_Pad1.30x1.75mm_HandSolder -> Resistor_SMD:R_0805_2012Metric
- R8: renamed from R9; footprint Resistor_SMD:R_1206_3216Metric_Pad1.30x1.75mm_HandSolder -> Resistor_SMD:R_0805_2012Metric
- R9: renamed from R10; footprint Resistor_SMD:R_1206_3216Metric_Pad1.30x1.75mm_HandSolder -> Resistor_SMD:R_0805_2012Metric
- renumbered C5 to C6, C6 to C7, C7 to C8, C8 to C9, JP11 to JP10, JP12 to JP11, JP13 to JP12, JP14 to JP13, JP15 to JP14, JP8 to JP7, JP9 to JP8, JP10 to JP9
Connections:
- net +3V3: now also C3.1, R10.1, R12.1
- net AUX_M1: now also U3.13 (LED7); no longer U3.19 (LED12)
- net AUX_M2: now also U3.12 (LED6); no longer U3.20 (LED13)
- net AUX_M3: now also U3.11 (LED5); no longer U3.21 (LED14)
- net CSENSE: now also U1.5 (AIN1); no longer U1.4 (AIN0)
- net GND: now also C3.2
- net M1: now also U3.15 (LED8); no longer U3.6 (LED0)
- net M10: now also U3.8 (LED2); no longer U3.16 (LED9)
- net M11: now also U3.7 (LED1); no longer U3.17 (LED10)
- net M12: now also U3.6 (LED0); no longer U3.18 (LED11)
- net M2: now also U3.16 (LED9); no longer U3.7 (LED1)
- net M3: now also U3.17 (LED10); no longer U3.8 (LED2)
- net M4: now also U3.18 (LED11); no longer U3.9 (LED3)
- net M5: now also U3.19 (LED12); no longer U3.10 (LED4)
- net M6: now also U3.20 (LED13); no longer U3.11 (LED5)
- net M7: now also U3.21 (LED14); no longer U3.12 (LED6)
- net M8: now also U3.22 (LED15); no longer U3.13 (LED7)
- net M9: now also U3.9 (LED3); no longer U3.15 (LED8)
- net SCL1: now also R10.2; no longer MOD1.5 (SCL), R5.2
- net SCL5: now also MOD1.5 (SCL), R5.2; no longer J14.3 (Pin_3)
- net SDA1: now also R12.2; no longer MOD1.4 (SDA), R2.2
- net SDA5: now also MOD1.4 (SDA), R2.2; no longer J14.2 (Pin_2)
- net VSENSE: now also U1.4 (AIN0); no longer U1.5 (AIN1)
- new net SCLXXX: J14.3 (Pin_3)
- new net SDAXXX: J14.2 (Pin_2)
Other:
- moved on the sheet: JP1, JP2, JP3, JP4, JP5, JP6, R1, R11, R13, R3, R4, R6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

Commit message: expansion board update
Parts:
- removed J7: Conn_02x03_Odd_Even, Connector_PinHeader_2.54mm:PinHeader_2x03_P2.54mm_Vertical, symbol Connector_Generic:Conn_02x03_Odd_Even
- removed JP1, JP2, JP3, JP4, JP5, JP6, JP7: SolderJumper_2_Open, Jumper:SolderJumper-2_P1.3mm_Open_Pad1.0x1.5mm, symbol Jumper:SolderJumper_2_Open
- removed JP11, JP8: Jumper_2_Open, Jumper:SolderJumper-2_P1.3mm_Open_Pad1.0x1.5mm, symbol Jumper:Jumper_2_Open
- removed R1, R11, R13, R20, R3, R4, R6, R7, R8, R9: 10k, Resistor_SMD:R_0805_2012Metric, symbol Device:R
- removed R24, R25, R26: 500Ω, Resistor_SMD:R_0805_2012Metric, symbol Device:R_Small_US
- added C10: C_Polarized, Capacitor_SMD:CP_Elec_10x10, symbol Device:C_Polarized
- added D1: D_Schottky, Diode_SMD:D_SMC, symbol Device:D_Schottky
- added JP1, JP4: Jumper_2_Open, Jumper:SolderJumper-2_P1.3mm_Open_Pad1.0x1.5mm, symbol Jumper:Jumper_2_Open
- added L1: L, Inductor_SMD:L_12x12mm_H6mm, symbol Device:L
- added R18: 3.9k, Resistor_SMD:R_0805_2012Metric, symbol Device:R_Small_US
- added R19: 1.21k, Resistor_SMD:R_0805_2012Metric, symbol Device:R_Small_US
- added R5, R6: 1.2k, Resistor_SMD:R_0805_2012Metric, symbol Device:R_Small_US
- added U12: LM2596S-5, Package_TO_SOT_SMD:TO-263-5_TabPin3, symbol Regulator_Switching:LM2596S-5
- U4: Address Address: 1001001 -> Address: 1001000
- renumbered C3 to C1, C1 to C2, C2 to C3, J11 to J10, J12 to J11, J13 to J12, J14 to J13, J15 to J14, J16 to J15, J9 to J7, J10 to J9, JP9 to JP2, JP10 to JP3, JP12 to JP5, JP13 to JP6, JP14 to JP7, R10 to R1, R17 to R10, R18 to R11, R19 to R12, R21 to R13, R22 to R14, R23 to R15, R27 to R16, R28 to R17, R12 to R2, R2 to R3, R5 to R4, R14 to R7, R15 to R8, R16 to R9, U3 to U2, U2 to U3
Connections:
- net GPIO27 is gone; now on net OUT4: J8.13 (GPIO27)
- net SCLXXX is gone; now on net SCL5: J13.3 (Pin_3)
- net SDAXXX is gone; now on net SDA5: J13.2 (Pin_2)
- net +3V3: now also J7.2 (Pin_2), J7.4 (Pin_4), J7.6 (Pin_6), R5.1, R6.1
- net +5V: now also C10.1, L1.1, R18.2, R19.1
- net +BATT: now also U12.1 (VIN)
- net FOOT1: now also JP1.2 (B)
- net FOOT2: now also JP2.2 (B); no longer JP3.2 (B)
- net FOOT3: now also JP3.2 (B); no longer JP2.2 (B)
- net FOOT4: now also JP4.2 (B)
- net GND: now also U1.1 (ADDR), U2.1 (A0), U2.2 (A1), U2.23 (~{OE}), U2.24 (A5), U2.25 (A6), U2.3 (A2), U2.4 (A3), U2.5 (A4), U4.1 (ADDR), C10.2, D1.2 (A), R19.2, U12.3 (GND), U12.5 (~{ON}/OFF)
- net NEOPIXEL: now also J8.19 (MOSI0/GPIO10); no longer J8.12 (GPIO18/PWM0)
- net OUT2: now also J8.7 (GCLK0/GPIO4); no longer J8.11 (GPIO17)
- net OUT3: now also J8.11 (GPIO17); no longer J8.35 (GPIO19/MISO1)
- net OUT4: no longer J8.38 (GPIO20/MOSI1)
- net OUT5: now also J8.18 (GPIO24); no longer J8.40 (GPIO21/SCLK1)
- net OUT6: now also J8.22 (GPIO25); no longer J8.18 (GPIO24)
- net OUT7: now also J8.21 (MISO0/GPIO9); no longer J8.22 (GPIO25)
- net SCL6: now also R6.2; no longer R15.2, U4.9 (SDA)
- net SDA6: now also R5.2; no longer R14.2, U4.10 (SCL)
- net SPI_CLK: now also J15.2 (Pin_2), J8.40 (GPIO21/SCLK1); no longer J15.4 (Pin_4), J8.23 (SCLK0/GPIO11)
- net SPI_CS: now also J8.12 (GPIO18/PWM0); no longer J8.24 (~{CE0}/GPIO8)
- net SPI_MISO: now also J15.4 (Pin_4), J8.35 (GPIO19/MISO1); no longer J15.2 (Pin_2), J8.21 (MISO0/GPIO9)
- net SPI_MOSI: now also J8.38 (GPIO20/MOSI1); no longer J8.19 (MOSI0/GPIO10)
- net at U5.10 (O7): now also J7.1 (Pin_1); no longer J7.5 (Pin_5)
- net at U5.12 (O5): now also J7.5 (Pin_5); no longer J7.1 (Pin_1)
- net +BATT-RAW: now reaches J2.2 (Pin_2), U3.1 (IP+), U3.2 (IP+)
- net SCL4: now reaches J8.26 (~{CE1}/GPIO7)
- net SCL4: now also R15.2, U4.9 (SDA)
- net GPIO26: no longer names the net of J8.37 (GPIO26)
- net GPIO26: now also JP1.1 (A)
- new net: D1.1 (K), L1.2, U12.2 (OUT)
- new net: R18.1, U12.4 (FB)
- new net: J8.23 (SCLK0/GPIO11), JP4.1 (A)
- new net SDA4: J8.24 (~{CE0}/GPIO8), R14.2, U4.10 (SCL)
- no-connect marks 10 -> 11
Other:
- note added: "Extra Power Connections"
- note removed: "Address Select"
- note removed: "Extra GPIO Breakout"
- note removed: "Power Connectors To/From DC-DC Convertors"
- moved on the sheet: C1, C2, C3, C4, C6, C7, C8, C9, H1, H2, H3, H4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

Commit message: expansion board update
Parts:
- removed R18: 3.9k, Resistor_SMD:R_0805_2012Metric, symbol Device:R_Small_US
- added D1: LED, LED_SMD:LED_0805_2012Metric, symbol Device:LED
- added R4: 10k, Resistor_SMD:R_0805_2012Metric, symbol Device:R_Small_US
- added RV1: 50k, General:Precision_pot, symbol Device:R_Potentiometer_Trim_US
- C7: renamed from C10; value C_Polarized -> 560uF
- L1: value L -> 22uH
- renumbered C9 to C10, C7 to C8, C8 to C9, D1 to D2, J11 to J10, J12 to J11, J8 to J12, J9 to J8, J10 to J9, R8 to R10, R10 to R11, R11 to R12, R12 to R13, R13 to R14, R14 to R15, R15 to R16, R19 to R17, R16 to R18, R17 to R19, R4 to R5, R5 to R6, R6 to R7, R7 to R8, U9 to U10, U10 to U12, U5 to U4, U4 to U5, U12 to U6, U6 to U8, U8 to U9
Connections:
- net +5V: now also RV1.1; no longer R17.1
- net +BATT-RAW: now also R4.2
- net GND: now also R17.1, D1.1 (K); no longer R17.2
- net at U6.4 (FB): now also R17.2, RV1.2, RV1.3
- new net: D1.2 (A), R4.1
Other:
- note added: "+5vDC Voltage Regulator for RPi4"
- note added: "Fixed voltage regulators require feedback resistance of zero ohms. Voltage divider present for adjustable regulator compatability."
- moved on the sheet: D2, H1, H2, H3, H4, H5, H6, R17
