Commit message: urdf update

File: quad_ws/src/quad_simulation/quad_simulation/src/urdf/zuko.urdf (robot description, URDF)
Before this commit: robot zuko, 20 links, 19 joints
Joints:
- joint back_left_lower_leg_rev_joint: axis 0 1 0 -> 0 -1 0; limit lower=-1.3962634015954636 upper=1.038470904936626 effort=4.0 velocity=4.0 -> lower=-3.141592653589793 upper=3.141592653589793 effort=4.0 velocity=4.0
- joint back_right_hip_rev_joint: axis -1 0 0 -> 1 0 0
- joint back_right_lower_leg_rev_joint: axis 0 1 0 -> 0 -1 0; limit lower=-1.3962634015954636 upper=1.038470904936626 effort=4.0 velocity=4.0 -> lower=-3.141592653589793 upper=3.141592653589793 effort=4.0 velocity=4.0
- joint front_left_lower_leg_rev_joint: axis 0 1 0 -> 0 -1 0; limit lower=-1.3962634015954636 upper=1.038470904936626 effort=4.0 velocity=4.0 -> lower=-3.141592653589793 upper=3.141592653589793 effort=4.0 velocity=4.0
- joint front_right_hip_rev_joint: axis 1 0 0 -> -1 0 0
- joint front_right_lower_leg_rev_joint: axis 0 1 0 -> 0 -1 0; limit lower=-1.3962634015954636 upper=1.038470904936626 effort=4.0 velocity=4.0 -> lower=-3.141592653589793 upper=3.141592653589793 effort=4.0 velocity=4.0

File: quad_ws/src/quad_udrf/urdf/zuko.urdf.xacro (robot description, xacro)
@@ -63,5 +63,5 @@
     <transmission name="${leg}_hip_joint_trans">
         <type>transmission_interface/SimpleTransmission</type>
-        <joint name="motor_${leg}_hip">
+        <joint name="${leg}_hip_rev_joint">
             <hardwareInterface>hardware_interface/EffortJointInterface</hardwareInterface>
         </joint>
@@ -73,5 +73,5 @@
     <transmission name="${leg}_upper_leg_joint_trans">
         <type>transmission_interface/SimpleTransmission</type>
-        <joint name="motor_${leg}_lower_leg">
+        <joint name="${leg}_lower_leg_rev_joint">
             <hardwareInterface>hardware_interface/EffortJointInterface</hardwareInterface>
         </joint>
@@ -83,5 +83,5 @@
     <transmission name="${leg}_lower_leg_joint_trans">
         <type>transmission_interface/SimpleTransmission</type>
-        <joint name="motor_${leg}_upper_leg">
+        <joint name="${leg}_upper_leg_rev_joint">
             <hardwareInterface>hardware_interface/EffortJointInterface</hardwareInterface>
         </joint>
@@ -259,6 +259,6 @@
 		<xacro:property name="upper_leg_upper_limit" value="${110 * pi/180}" />
 		<xacro:property name="upper_leg_lower_limit" value="${0 * pi/180}" />
-		<xacro:property name="lower_leg_upper_limit" value="${59.5 * pi/180}" />
-		<xacro:property name="lower_leg_lower_limit" value="${-80 * pi/180}" />
+		<xacro:property name="lower_leg_upper_limit" value="${180 * pi/180}" />
+		<xacro:property name="lower_leg_lower_limit" value="${-180 * pi/180}" />
 	<!-- FRONT LEFT -->
 		<xacro:mesh_link name="front_left_hip_link"
@@ -315,5 +315,5 @@
 				    child="front_left_upper_leg_link" />
 		<xacro:mesh_link name="front_left_lower_leg_link"
-					origin_rpy="${pi/2} 0 ${pi}"
+					origin_rpy="${pi/2} ${pi/2} ${pi}"
 					origin_xyz="0 -${upper_leg_origin_offset_to_center_of_leg} 0"
 					i_rpy="0 0 0"
@@ -329,5 +329,5 @@
 		<xacro:rev_joint name="front_left_lower_leg_rev_joint"
 					type="revolute"
-				    axis_xyz="0 1 0"
+				    axis_xyz="0 -1 0"
 				    origin_rpy="0 0 ${pi}"
 					origin_xyz="${0} ${0} -${upper_leg_length_between_joints}"
@@ -356,5 +356,5 @@
 		<xacro:rev_joint name="front_right_hip_rev_joint"
 				type="revolute"
-			    axis_xyz="1 0 0"
+			    axis_xyz="-1 0 0"
 			    origin_rpy="0 0 ${pi}"
 				origin_xyz="${servo_flange_protrusion_from_center_distance} -0.0455 0"
@@ -394,10 +394,10 @@
 				    child="front_right_upper_leg_link" />
 		<xacro:mesh_link name="front_right_lower_leg_link"
-					origin_rpy="${pi/2} 0 ${pi}"
+					origin_rpy="${pi/2} ${pi/2}  ${pi}"
 					origin_xyz="0 ${upper_leg_origin_offset_to_center_of_leg} 0"
 					i_rpy="0 0 0"
 					i_xyz="0 0 0"
 					mass="0.6"
-					c_xyz="0 0 0"
+					c_xyz="0 0 -0.06"
 					length="0"
 					width="0"
@@ -408,5 +408,5 @@
 		<xacro:rev_joint name="front_right_lower_leg_rev_joint"
 					type="revolute"
-				    axis_xyz="0 1 0"
+				    axis_xyz="0 -1 0"
 				    origin_rpy="0 0 ${pi}"
 					origin_xyz="${0} ${0} -${upper_leg_length_between_joints}"
@@ -473,5 +473,5 @@
 				    child="back_left_upper_leg_link" />
 		<xacro:mesh_link name="back_left_lower_leg_link"
-					origin_rpy="${pi/2} 0 ${pi}"
+					origin_rpy="${pi/2} ${pi/2} ${pi}"
 					origin_xyz="0 -${upper_leg_origin_offset_to_center_of_leg} 0"
 					i_rpy="0 0 0"
@@ -487,5 +487,5 @@
 		<xacro:rev_joint name="back_left_lower_leg_rev_joint"
 					type="revolute"
-				    axis_xyz="0 1 0"
+				    axis_xyz="0 -1 0"
 				    origin_rpy="0 0 ${pi}"
 					origin_xyz="${0} ${0} -${upper_leg_length_between_joints}"
@@ -514,5 +514,5 @@
 		<xacro:rev_joint name="back_right_hip_rev_joint"
 				type="revolute"
-			    axis_xyz="-1 0 0"
+			    axis_xyz="1 0 0"
 			    origin_rpy="0 0 0"
 				origin_xyz="-${servo_flange_protrusion_from_center_distance} -0.0455 0"
@@ -552,10 +552,10 @@
 				    child="back_right_upper_leg_link" />
 		<xacro:mesh_link name="back_right_lower_leg_link"
-					origin_rpy="${pi/2} 0 ${pi}"
+					origin_rpy="${pi/2} ${pi/2} ${pi}"
 					origin_xyz="0 ${upper_leg_origin_offset_to_center_of_leg} 0"
 					i_rpy="0 0 0"
 					i_xyz="0 0 0"
 					mass="0.6"
-					c_xyz="0 0 0"
+					c_xyz="0  -0.06 0"
 					length="0"
 					width="0"
@@ -566,5 +566,5 @@
 		<xacro:rev_joint name="back_right_lower_leg_rev_joint"
 					type="revolute"
-				    axis_xyz="0 1 0"
+				    axis_xyz="0 -1 0"
 				    origin_rpy="0 0 ${pi}"
 					origin_xyz="${0} ${0} -${upper_leg_length_between_joints}"

Commit message: frame param update / doc update

File: quad_ws/src/quad_simulation/quad_simulation/src/urdf/zuko.urdf (robot description, URDF)
Before this commit: robot zuko, 20 links, 19 joints
Links:
- link back_left_hip_link: geometry collision mesh filename=package://stl/hip_back.stl scale=1 1 1; visual mesh filename=package://stl/hip_back.stl scale=1 1 1
- link back_left_lower_leg_link: geometry collision mesh filename=package://stl/lower_leg.stl scale=1 1 1; visual mesh filename=package://stl/lower_leg.stl scale=1 1 1
- link back_left_upper_leg_link: geometry collision mesh filename=package://stl/upper_leg.stl scale=1 1 1; visual mesh filename=package://stl/upper_leg.stl scale=1 1 1
- link back_right_hip_link: geometry collision mesh filename=package://stl/hip_back.stl scale=1 -1 1; visual mesh filename=package://stl/hip_back.stl scale=1 -1 1
- link back_right_lower_leg_link: geometry collision mesh filename=package://stl/lower_leg.stl scale=1 1 -1; visual mesh filename=package://stl/lower_leg.stl scale=1 1 -1
- link back_right_upper_leg_link: geometry collision mesh filename=package://stl/upper_leg.stl scale=1 1 1; visual mesh filename=package://stl/upper_leg.stl scale=1 1 1
- link base_link: geometry collision mesh filename=package://stl/center_front.stl scale=1 1 1; visual mesh filename=package://stl/center_front.stl scale=1 1 1
- link bridge_back_link: geometry collision mesh filename=package://stl/bridge_back.stl scale=1 1 1; visual mesh filename=package://stl/bridge_back.stl scale=1 1 1
- link bridge_front_link: geometry collision mesh filename=package://stl/bridge_front.stl scale=1 1 1; visual mesh filename=package://stl/bridge_front.stl scale=1 1 1
- link butt_link: geometry collision mesh filename=package://stl/butt.stl scale=1 1 1; visual mesh filename=package://stl/butt.stl scale=1 1 1
- link center_back_link: geometry collision mesh filename=package://stl/center_back.stl scale=1 1 1; visual mesh filename=package://stl/center_back.stl scale=1 1 1
- link face_link: geometry collision mesh filename=package://stl/face.stl scale=1 1 1; visual mesh filename=package://stl/face.stl scale=1 1 1
- link front_left_hip_link: geometry collision mesh filename=package://stl/hip_front.stl scale=1 1 1; visual mesh filename=package://stl/hip_front.stl scale=1 1 1
- link front_left_lower_leg_link: geometry collision mesh filename=package://stl/lower_leg.stl scale=1 1 1; visual mesh filename=package://stl/lower_leg.stl scale=1 1 1
- link front_left_upper_leg_link: geometry collision mesh filename=package://stl/upper_leg.stl scale=1 1 1; visual mesh filename=package://stl/upper_leg.stl scale=1 1 1
- link front_right_hip_link: geometry collision mesh filename=package://stl/hip_front.stl scale=1 -1 1; visual mesh filename=package://stl/hip_front.stl scale=1 -1 1
- link front_right_lower_leg_link: geometry collision mesh filename=package://stl/lower_leg.stl scale=1 1 -1; visual mesh filename=package://stl/lower_leg.stl scale=1 1 -1
- link front_right_upper_leg_link: geometry collision mesh filename=package://stl/upper_leg.stl scale=1 1 1; visual mesh filename=package://stl/upper_leg.stl scale=1 1 1
- link side_left_link: geometry collision mesh filename=package://stl/side_left.stl scale=1 1 1; visual mesh filename=package://stl/side_left.stl scale=1 1 1
- link side_right_link: geometry collision mesh filename=package://stl/side_right.stl scale=1 1 1; visual mesh filename=package://stl/side_right.stl scale=1 1 1
Joints:
- joint back_left_upper_leg_rev_joint: limit lower=0.0 upper=1.9198621771937625 effort=4.0 velocity=4.0 -> lower=-3.141592653589793 upper=3.141592653589793 effort=4.0 velocity=4.0
- joint back_right_upper_leg_rev_joint: limit lower=0.0 upper=1.9198621771937625 effort=4.0 velocity=4.0 -> lower=-3.141592653589793 upper=3.141592653589793 effort=4.0 velocity=4.0
- joint center_back_joint: origin xyz=-0.18399999999999997 0 0 rpy=0 0 0 -> xyz=-0.16599999999999998 0 0 rpy=0 0 0
- joint front_left_upper_leg_rev_joint: limit lower=0.0 upper=1.9198621771937625 effort=4.0 velocity=4.0 -> lower=-3.141592653589793 upper=3.141592653589793 effort=4.0 velocity=4.0
- joint front_right_upper_leg_rev_joint: limit lower=0.0 upper=1.9198621771937625 effort=4.0 velocity=4.0 -> lower=-3.141592653589793 upper=3.141592653589793 effort=4.0 velocity=4.0

File: quad_ws/src/quad_udrf/urdf/zuko.urdf.xacro (robot description, xacro)
@@ -25,5 +25,6 @@
 		<origin rpy="${origin_rpy}" xyz="${c_xyz}" />
 		<geometry>
-		  <box size="${length} ${width} ${height}" />
+		  <!--<box size="${length} ${width} ${height}" />-->
+		  <mesh filename="${meshfile}" scale="${meshscale}"/>
 		</geometry>
 	  </collision>
@@ -218,5 +219,5 @@
 			type="fixed"
 			origin_rpy="0 0 0"
-			origin_xyz="-${side_length + center_thickness + center_thickness} 0 0"
+			origin_xyz="-${side_length + center_thickness} 0 0"
 			parent="base_link"
 			child="center_back_link"/>
@@ -255,10 +256,15 @@
 		<xacro:property name="upper_leg_length_between_joints" value="${0.100}" />
 	<!-- Limits -->
+	<!-- No effective limits in the URDF model as they are defined elsewhere,
+	 and we want to see if the kinematics don't breach the intended limits -->
 		<xacro:property name="hip_upper_limit" value="${30 * pi/180}" />
 		<xacro:property name="hip_lower_limit" value="${-30 * pi/180}" />
-		<xacro:property name="upper_leg_upper_limit" value="${110 * pi/180}" />
-		<xacro:property name="upper_leg_lower_limit" value="${0 * pi/180}" />
+		<xacro:property name="upper_leg_upper_limit" value="${180 * pi/180}" />
+		<xacro:property name="upper_leg_lower_limit" value="${-180 * pi/180}" />
 		<xacro:property name="lower_leg_upper_limit" value="${180 * pi/180}" />
 		<xacro:property name="lower_leg_lower_limit" value="${-180 * pi/180}" />
+<!--
+<xacro:property name="path" value="package://stl" />
+-->
 	<!-- FRONT LEFT -->
 		<xacro:mesh_link name="front_left_hip_link"
@@ -320,5 +326,5 @@
 					i_xyz="0 0 0"
 					mass="0.6"
-					c_xyz="0 0 0"
+					c_xyz="0 -${upper_leg_origin_offset_to_center_of_leg} 0"
 					length="0"
 					width="0"
@@ -399,5 +405,5 @@
 					i_xyz="0 0 0"
 					mass="0.6"
-					c_xyz="0 0 -0.06"
+					c_xyz="0 ${upper_leg_origin_offset_to_center_of_leg} 0"
 					length="0"
 					width="0"
@@ -478,5 +484,5 @@
 					i_xyz="0 0 0"
 					mass="0.6"
-					c_xyz="0 0 0"
+					c_xyz="0 -${upper_leg_origin_offset_to_center_of_leg} 0"
 					length="0"
 					width="0"
@@ -557,8 +563,8 @@
 					i_xyz="0 0 0"
 					mass="0.6"
-					c_xyz="0  -0.06 0"
-					length="0"
-					width="0"
-					height="0"
+					c_xyz="0 ${upper_leg_origin_offset_to_center_of_leg} 0"
+					length="0.1125"
+					width="0.25"
+					height="0.25"
 					matname="brown"
 					meshfile="package://stl/lower_leg.stl"
