Commit message: zuko URDF first time in sim gym

File: quad_ws/src/quad_simulation/quad_simulation/src/urdf/quad.urdf (robot description, URDF)
Before this commit: robot spot, 25 links, 24 joints
Links:
- removed link back
- removed link back_bracket
- removed link back_left_foot
- removed link back_left_hip
- removed link back_left_lower_leg
- removed link back_left_upper_leg
- removed link back_right_foot
- removed link back_right_hip
- removed link back_right_lower_leg
- removed link back_right_upper_leg
- removed link base_inertia
- removed link battery
- removed link chassis_left
- removed link chassis_right
- removed link front
- removed link front_bracket
- removed link front_left_foot
- removed link front_left_hip
- removed link front_left_lower_leg
- removed link front_left_upper_leg
- removed link front_right_foot
- removed link front_right_hip
- removed link front_right_lower_leg
- removed link front_right_upper_leg
- added link back_left_hip_link, mass 0.6; collision box size=0 0 0; visual mesh filename=package://quad_urdf/stl/hip_back.stl scale=1 1 1
- added link back_left_lower_leg_link, mass 0.6; collision box size=0 0 0; visual mesh filename=package://quad_urdf/stl/lower_leg.stl scale=1 1 1
- added link back_left_upper_leg_link, mass 0.6; collision box size=0 0 0; visual mesh filename=package://quad_urdf/stl/upper_leg.stl scale=1 1 1
- added link back_right_hip_link, mass 0.6; collision box size=0 0 0; visual mesh filename=package://quad_urdf/stl/hip_back.stl scale=1 -1 1
- added link back_right_lower_leg_link, mass 0.6; collision box size=0 0 0; visual mesh filename=package://quad_urdf/stl/lower_leg.stl scale=1 1 -1
- added link back_right_upper_leg_link, mass 0.6; collision box size=0 0 0; visual mesh filename=package://quad_urdf/stl/upper_leg.stl scale=1 1 1
- added link bridge_back_link, mass 0.6; collision box size=0 0 0; visual mesh filename=package://quad_urdf/stl/bridge_back.stl scale=1 1 1
- added link bridge_front_link, mass 0.6; collision box size=0 0 0; visual mesh filename=package://quad_urdf/stl/bridge_front.stl scale=1 1 1
- added link butt_link, mass 0.6; collision box size=0 0 0; visual mesh filename=package://quad_urdf/stl/butt.stl scale=1 1 1
- added link center_back_link, mass 0.6; collision box size=0 0 0; visual mesh filename=package://quad_urdf/stl/center_back.stl scale=1 1 1
- added link face_link, mass 0.6; collision box size=0 0 0; visual mesh filename=package://quad_urdf/stl/face.stl scale=1 1 1
- added link front_left_hip_link, mass 0.6; collision box size=0 0 0; visual mesh filename=package://quad_urdf/stl/hip_front.stl scale=1 1 1
- added link front_left_lower_leg_link, mass 0.6; collision box size=0 0 0; visual mesh filename=package://quad_urdf/stl/lower_leg.stl scale=1 1 1
- added link front_left_upper_leg_link, mass 0.6; collision box size=0 0 0; visual mesh filename=package://quad_urdf/stl/upper_leg.stl scale=1 1 1
- added link front_right_hip_link, mass 0.6; collision box size=0 0 0; visual mesh filename=package://quad_urdf/stl/hip_front.stl scale=1 -1 1
- added link front_right_lower_leg_link, mass 0.6; collision box size=0 0 0; visual mesh filename=package://quad_urdf/stl/lower_leg.stl scale=1 1 -1
- added link front_right_upper_leg_link, mass 0.6; collision box size=0 0 0; visual mesh filename=package://quad_urdf/stl/upper_leg.stl scale=1 1 1
- added link side_left_link, mass 0.6; collision box size=0 0 0; visual mesh filename=package://quad_urdf/stl/side_left.stl scale=1 1 1
- added link side_right_link, mass 0.6; collision box size=0 0 0; visual mesh filename=package://quad_urdf/stl/side_right.stl scale=1 1 1
- link base_link: mass None -> 0.6; geometry collision box size=0 0 0; visual mesh filename=package://quad_urdf/stl/center_front.stl scale=1 1 1
Joints:
- removed joint back_left_leg_foot
- removed joint back_right_leg_foot
- removed joint base_back
- removed joint base_back_bracket
- removed joint base_base
- removed joint base_battery
- removed joint base_front
- removed joint base_front_bracket
- removed joint base_left
- removed joint base_right
- removed joint front_left_leg_foot
- removed joint front_right_leg_foot
- removed joint motor_back_left_hip
- removed joint motor_back_left_lower_leg
- removed joint motor_back_left_upper_leg
- removed joint motor_back_right_hip
- removed joint motor_back_right_lower_leg
- removed joint motor_back_right_upper_leg
- removed joint motor_front_left_hip
- removed joint motor_front_left_lower_leg
- removed joint motor_front_left_upper_leg
- removed joint motor_front_right_hip
- removed joint motor_front_right_lower_leg
- removed joint motor_front_right_upper_leg
- added joint back_left_hip_rev_joint: type revolute, parent center_back_link, child back_left_hip_link, origin xyz=-0.002 0.0455 0 rpy=0 0 0, axis 1 0 0, limit lower=-0.5235987755982988 upper=0.5235987755982988 effort=4.0 velocity=4.0
- added joint back_left_lower_leg_rev_joint: type revolute, parent back_left_upper_leg_link, child back_left_lower_leg_link, origin xyz=0 0 -0.1 rpy=0 0 3.141592653589793, axis 0 1 0, limit lower=-1.3962634015954636 upper=1.038470904936626 effort=4.0 velocity=4.0
- added joint back_left_upper_leg_rev_joint: type revolute, parent back_left_hip_link, child back_left_upper_leg_link, origin xyz=-0.035500000000000004 0.03175 0 rpy=0 0 0, axis 0 1 0, limit lower=0.0 upper=1.9198621771937625 effort=4.0 velocity=4.0
- added joint back_right_hip_rev_joint: type revolute, parent center_back_link, child back_right_hip_link, origin xyz=-0.002 -0.0455 0 rpy=0 0 0, axis -1 0 0, limit lower=-0.5235987755982988 upper=0.5235987755982988 effort=4.0 velocity=4.0
- added joint back_right_lower_leg_rev_joint: type revolute, parent back_right_upper_leg_link, child back_right_lower_leg_link, origin xyz=0 0 -0.1 rpy=0 0 3.141592653589793, axis 0 1 0, limit lower=-1.3962634015954636 upper=1.038470904936626 effort=4.0 velocity=4.0
- added joint back_right_upper_leg_rev_joint: type revolute, parent back_right_hip_link, child back_right_upper_leg_link, origin xyz=-0.035500000000000004 -0.03175 0 rpy=0 0 0, axis 0 1 0, limit lower=0.0 upper=1.9198621771937625 effort=4.0 velocity=4.0
- added joint bridge_back_joint: type fixed, parent center_back_link, child bridge_back_link, origin xyz=0 0 -0.011 rpy=0 0 0
- added joint bridge_front_joint: type fixed, parent base_link, child bridge_front_link, origin xyz=0.0535 0 -0.011 rpy=0 0  0
- added joint butt_joint: type fixed, parent bridge_back_link, child butt_link, origin xyz=-0.0535 0 0 rpy=0 0 0
- added joint center_back_joint: type fixed, parent base_link, child center_back_link, origin xyz=-0.18399999999999997 0 0 rpy=0 0 0
- added joint face_joint: type fixed, parent bridge_front_link, child face_link, origin xyz=0 0 0 rpy=0 0 0
- added joint front_left_hip_rev_joint: type revolute, parent base_link, child front_left_hip_link, origin xyz=0.002 0.0455 0 rpy=0 0 3.141592653589793, axis -1 0 0, limit lower=-0.5235987755982988 upper=0.5235987755982988 effort=4.0 velocity=4.0
- added joint front_left_lower_leg_rev_joint: type revolute, parent front_left_upper_leg_link, child front_left_lower_leg_link, origin xyz=0 0 -0.1 rpy=0 0 3.141592653589793, axis 0 1 0, limit lower=-1.3962634015954636 upper=1.038470904936626 effort=4.0 velocity=4.0
- added joint front_left_upper_leg_rev_joint: type revolute, parent front_left_hip_link, child front_left_upper_leg_link, origin xyz=-0.0145 -0.03175 0 rpy=0 0 3.141592653589793, axis 0 1 0, limit lower=0.0 upper=1.9198621771937625 effort=4.0 velocity=4.0
- added joint front_right_hip_rev_joint: type revolute, parent base_link, child front_right_hip_link, origin xyz=0.002 -0.0455 0 rpy=0 0 3.141592653589793, axis 1 0 0, limit lower=-0.5235987755982988 upper=0.5235987755982988 effort=4.0 velocity=4.0
- added joint front_right_lower_leg_rev_joint: type revolute, parent front_right_upper_leg_link, child front_right_lower_leg_link, origin xyz=0 0 -0.1 rpy=0 0 3.141592653589793, axis 0 1 0, limit lower=-1.3962634015954636 upper=1.038470904936626 effort=4.0 velocity=4.0
- added joint front_right_upper_leg_rev_joint: type revolute, parent front_right_hip_link, child front_right_upper_leg_link, origin xyz=-0.0145 0.03175 0 rpy=0 0 3.141592653589793, axis 0 1 0, limit lower=0.0 upper=1.9198621771937625 effort=4.0 velocity=4.0
- added joint side_left_joint: type fixed, parent base_link, child side_left_link, origin xyz=-0.16599999999999998 0.060 0.015 rpy=0 0 0
- added joint side_right_joint: type fixed, parent base_link, child side_right_link, origin xyz=-0.018 -0.060 0.015 rpy=0 0 0

File: quad_ws/src/quad_simulation/quad_simulation/src/urdf/zuko.urdf (robot description, URDF)
Before this commit: robot zuko, 20 links, 19 joints
Links:
- link back_left_hip_link: geometry collision box size=0 0 0; visual mesh filename=package://stl/hip_back.stl scale=1 1 1
- link back_left_lower_leg_link: geometry collision box size=0 0 0; visual mesh filename=package://stl/lower_leg.stl scale=1 1 1
- link back_left_upper_leg_link: geometry collision box size=0 0 0; visual mesh filename=package://stl/upper_leg.stl scale=1 1 1
- link back_right_hip_link: geometry collision box size=0 0 0; visual mesh filename=package://stl/hip_back.stl scale=1 -1 1
- link back_right_lower_leg_link: geometry collision box size=0 0 0; visual mesh filename=package://stl/lower_leg.stl scale=1 1 -1
- link back_right_upper_leg_link: geometry collision box size=0 0 0; visual mesh filename=package://stl/upper_leg.stl scale=1 1 1
- link base_link: geometry collision box size=0 0 0; visual mesh filename=package://stl/center_front.stl scale=1 1 1
- link bridge_back_link: geometry collision box size=0 0 0; visual mesh filename=package://stl/bridge_back.stl scale=1 1 1
- link bridge_front_link: geometry collision box size=0 0 0; visual mesh filename=package://stl/bridge_front.stl scale=1 1 1
- link butt_link: geometry collision box size=0 0 0; visual mesh filename=package://stl/butt.stl scale=1 1 1
- link center_back_link: geometry collision box size=0 0 0; visual mesh filename=package://stl/center_back.stl scale=1 1 1
- link face_link: geometry collision box size=0 0 0; visual mesh filename=package://stl/face.stl scale=1 1 1
- link front_left_hip_link: geometry collision box size=0 0 0; visual mesh filename=package://stl/hip_front.stl scale=1 1 1
- link front_left_lower_leg_link: geometry collision box size=0 0 0; visual mesh filename=package://stl/lower_leg.stl scale=1 1 1
- link front_left_upper_leg_link: geometry collision box size=0 0 0; visual mesh filename=package://stl/upper_leg.stl scale=1 1 1
- link front_right_hip_link: geometry collision box size=0 0 0; visual mesh filename=package://stl/hip_front.stl scale=1 -1 1
- link front_right_lower_leg_link: geometry collision box size=0 0 0; visual mesh filename=package://stl/lower_leg.stl scale=1 1 -1
- link front_right_upper_leg_link: geometry collision box size=0 0 0; visual mesh filename=package://stl/upper_leg.stl scale=1 1 1
- link side_left_link: geometry collision box size=0 0 0; visual mesh filename=package://stl/side_left.stl scale=1 1 1
- link side_right_link: geometry collision box size=0 0 0; visual mesh filename=package://stl/side_right.stl scale=1 1 1

File: quad_ws/src/quad_udrf/urdf/zuko.urdf.xacro (robot description, xacro)
@@ -109,5 +109,5 @@
 		height="0"
 		matname="brown"
-		meshfile="package://quad_urdf/stl/center_front.stl"
+		meshfile="package://stl/center_front.stl"
 		meshscale="1 1 1" />
 	<xacro:mesh_link name="side_left_link"
@@ -122,5 +122,5 @@
 		height="0"
 		matname="brown"
-		meshfile="package://quad_urdf/stl/side_left.stl"
+		meshfile="package://stl/side_left.stl"
 		meshscale="1 1 1" />
 	<xacro:mesh_link name="side_right_link"
@@ -135,5 +135,5 @@
 		height="0"
 		matname="brown"
-		meshfile="package://quad_urdf/stl/side_right.stl"
+		meshfile="package://stl/side_right.stl"
 		meshscale="1 1 1" />
 	<xacro:mesh_link name="center_back_link"
@@ -148,5 +148,5 @@
 		height="0"
 		matname="brown"
-		meshfile="package://quad_urdf/stl/center_back.stl"
+		meshfile="package://stl/center_back.stl"
 		meshscale="1 1 1" />
 	<xacro:mesh_link name="bridge_front_link"
@@ -161,5 +161,5 @@
 		height="0"
 		matname="white"
-		meshfile="package://quad_urdf/stl/bridge_front.stl"
+		meshfile="package://stl/bridge_front.stl"
 		meshscale="1 1 1" />
 	<xacro:mesh_link name="bridge_back_link"
@@ -174,5 +174,5 @@
 		height="0"
 		matname="white"
-		meshfile="package://quad_urdf/stl/bridge_back.stl"
+		meshfile="package://stl/bridge_back.stl"
 		meshscale="1 1 1" />
 	<xacro:mesh_link name="face_link"
@@ -187,5 +187,5 @@
 		height="0"
 		matname="brown"
-		meshfile="package://quad_urdf/stl/face.stl"
+		meshfile="package://stl/face.stl"
 		meshscale="1 1 1" />
 	<xacro:mesh_link name="butt_link"
@@ -200,5 +200,5 @@
 		height="0"
 		matname="brown"
-		meshfile="package://quad_urdf/stl/butt.stl"
+		meshfile="package://stl/butt.stl"
 		meshscale="1 1 1" />
 <!-- STATIC Joints -->
@@ -273,5 +273,5 @@
 				height="0"
 				matname="white"
-				meshfile="package://quad_urdf/stl/hip_front.stl"
+				meshfile="package://stl/hip_front.stl"
 				meshscale="1 1 1" />
 		<xacro:rev_joint name="front_left_hip_rev_joint"
@@ -299,5 +299,5 @@
 					height="0"
 					matname="brown"
-					meshfile="package://quad_urdf/stl/upper_leg.stl"
+					meshfile="package://stl/upper_leg.stl"
 					meshscale="1 1 1" />
 		<xacro:rev_joint name="front_left_upper_leg_rev_joint"
@@ -325,5 +325,5 @@
 					height="0"
 					matname="brown"
-					meshfile="package://quad_urdf/stl/lower_leg.stl"
+					meshfile="package://stl/lower_leg.stl"
 					meshscale="1 1 1" />
 		<xacro:rev_joint name="front_left_lower_leg_rev_joint"
@@ -352,5 +352,5 @@
 				height="0"
 				matname="white"
-				meshfile="package://quad_urdf/stl/hip_front.stl"
+				meshfile="package://stl/hip_front.stl"
 				meshscale="1 -1 1" />
 		<xacro:rev_joint name="front_right_hip_rev_joint"
@@ -378,5 +378,5 @@
 					height="0"
 					matname="brown"
-					meshfile="package://quad_urdf/stl/upper_leg.stl"
+					meshfile="package://stl/upper_leg.stl"
 					meshscale="1 1 1" />
 		<xacro:rev_joint name="front_right_upper_leg_rev_joint"
@@ -404,5 +404,5 @@
 					height="0"
 					matname="brown"
-					meshfile="package://quad_urdf/stl/lower_leg.stl"
+					meshfile="package://stl/lower_leg.stl"
 					meshscale="1 1 -1" />
 		<xacro:rev_joint name="front_right_lower_leg_rev_joint"
@@ -431,5 +431,5 @@
 				height="0"
 				matname="white"
-				meshfile="package://quad_urdf/stl/hip_back.stl"
+				meshfile="package://stl/hip_back.stl"
 				meshscale="1 1 1" />
 		<xacro:rev_joint name="back_left_hip_rev_joint"
@@ -457,5 +457,5 @@
 					height="0"
 					matname="brown"
-					meshfile="package://quad_urdf/stl/upper_leg.stl"
+					meshfile="package://stl/upper_leg.stl"
 					meshscale="1 1 1" />
 		<xacro:rev_joint name="back_left_upper_leg_rev_joint"
@@ -483,5 +483,5 @@
 					height="0"
 					matname="brown"
-					meshfile="package://quad_urdf/stl/lower_leg.stl"
+					meshfile="package://stl/lower_leg.stl"
 					meshscale="1 1 1" />
 		<xacro:rev_joint name="back_left_lower_leg_rev_joint"
@@ -510,5 +510,5 @@
 				height="0"
 				matname="white"
-				meshfile="package://quad_urdf/stl/hip_back.stl"
+				meshfile="package://stl/hip_back.stl"
 				meshscale="1 -1 1" />
 		<xacro:rev_joint name="back_right_hip_rev_joint"
@@ -536,5 +536,5 @@
 					height="0"
 					matname="brown"
-					meshfile="package://quad_urdf/stl/upper_leg.stl"
+					meshfile="package://stl/upper_leg.stl"
 					meshscale="1 1 1" />
 		<xacro:rev_joint name="back_right_upper_leg_rev_joint"
@@ -562,5 +562,5 @@
 					height="0"
 					matname="brown"
-					meshfile="package://quad_urdf/stl/lower_leg.stl"
+					meshfile="package://stl/lower_leg.stl"
 					meshscale="1 1 -1" />
 		<xacro:rev_joint name="back_right_lower_leg_rev_joint"
