Commit message: added joy index to gamepad as param

File: quad_ws/src/quad_simulation/quad_simulation/src/urdf/quad.urdf (robot description, URDF)
Before this commit: robot zuko, 20 links, 19 joints
Links:
- link back_left_hip_link: geometry collision mesh filename=package://stl/hip_back.stl scale=1 1 1; visual mesh filename=package://stl/hip_back.stl scale=1 1 1
- link back_left_lower_leg_link: geometry collision mesh filename=package://stl/lower_leg.stl scale=1 1 1; visual mesh filename=package://stl/lower_leg.stl scale=1 1 1
- link back_left_upper_leg_link: geometry collision mesh filename=package://stl/upper_leg.stl scale=1 1 1; visual mesh filename=package://stl/upper_leg.stl scale=1 1 1
- link back_right_hip_link: geometry collision mesh filename=package://stl/hip_back.stl scale=1 -1 1; visual mesh filename=package://stl/hip_back.stl scale=1 -1 1
- link back_right_lower_leg_link: geometry collision mesh filename=package://stl/lower_leg.stl scale=1 1 -1; visual mesh filename=package://stl/lower_leg.stl scale=1 1 -1
- link back_right_upper_leg_link: geometry collision mesh filename=package://stl/upper_leg.stl scale=1 1 1; visual mesh filename=package://stl/upper_leg.stl scale=1 1 1
- link base_link: geometry collision mesh filename=package://stl/center_front.stl scale=1 1 1; visual mesh filename=package://stl/center_front.stl scale=1 1 1
- link bridge_back_link: geometry collision mesh filename=package://stl/bridge_back.stl scale=1 1 1; visual mesh filename=package://stl/bridge_back.stl scale=1 1 1
- link bridge_front_link: geometry collision mesh filename=package://stl/bridge_front.stl scale=1 1 1; visual mesh filename=package://stl/bridge_front.stl scale=1 1 1
- link butt_link: geometry collision mesh filename=package://stl/butt.stl scale=1 1 1; visual mesh filename=package://stl/butt.stl scale=1 1 1
- link center_back_link: geometry collision mesh filename=package://stl/center_back.stl scale=1 1 1; visual mesh filename=package://stl/center_back.stl scale=1 1 1
- link face_link: geometry collision mesh filename=package://stl/face.stl scale=1 1 1; visual mesh filename=package://stl/face.stl scale=1 1 1
- link front_left_hip_link: geometry collision mesh filename=package://stl/hip_front.stl scale=1 1 1; visual mesh filename=package://stl/hip_front.stl scale=1 1 1
- link front_left_lower_leg_link: geometry collision mesh filename=package://stl/lower_leg.stl scale=1 1 1; visual mesh filename=package://stl/lower_leg.stl scale=1 1 1
- link front_left_upper_leg_link: geometry collision mesh filename=package://stl/upper_leg.stl scale=1 1 1; visual mesh filename=package://stl/upper_leg.stl scale=1 1 1
- link front_right_hip_link: geometry collision mesh filename=package://stl/hip_front.stl scale=1 -1 1; visual mesh filename=package://stl/hip_front.stl scale=1 -1 1
- link front_right_lower_leg_link: geometry collision mesh filename=package://stl/lower_leg.stl scale=1 1 -1; visual mesh filename=package://stl/lower_leg.stl scale=1 1 -1
- link front_right_upper_leg_link: geometry collision mesh filename=package://stl/upper_leg.stl scale=1 1 1; visual mesh filename=package://stl/upper_leg.stl scale=1 1 1
- link side_left_link: geometry collision mesh filename=package://stl/side_left.stl scale=1 1 1; visual mesh filename=package://stl/side_left.stl scale=1 1 1
- link side_right_link: geometry collision mesh filename=package://stl/side_right.stl scale=1 1 1; visual mesh filename=package://stl/side_right.stl scale=1 1 1
Joints:
- joint back_left_lower_leg_rev_joint: axis 0 1 0 -> 0 -1 0; limit lower=-1.3962634015954636 upper=1.038470904936626 effort=4.0 velocity=4.0 -> lower=-3.141592653589793 upper=3.141592653589793 effort=4.0 velocity=4.0
- joint back_left_upper_leg_rev_joint: limit lower=0.0 upper=1.9198621771937625 effort=4.0 velocity=4.0 -> lower=-3.141592653589793 upper=3.141592653589793 effort=4.0 velocity=4.0
- joint back_right_hip_rev_joint: axis -1 0 0 -> 1 0 0
- joint back_right_lower_leg_rev_joint: axis 0 1 0 -> 0 -1 0; limit lower=-1.3962634015954636 upper=1.038470904936626 effort=4.0 velocity=4.0 -> lower=-3.141592653589793 upper=3.141592653589793 effort=4.0 velocity=4.0
- joint back_right_upper_leg_rev_joint: limit lower=0.0 upper=1.9198621771937625 effort=4.0 velocity=4.0 -> lower=-3.141592653589793 upper=3.141592653589793 effort=4.0 velocity=4.0
- joint center_back_joint: origin xyz=-0.18399999999999997 0 0 rpy=0 0 0 -> xyz=-0.16599999999999998 0 0 rpy=0 0 0
- joint front_left_lower_leg_rev_joint: axis 0 1 0 -> 0 -1 0; limit lower=-1.3962634015954636 upper=1.038470904936626 effort=4.0 velocity=4.0 -> lower=-3.141592653589793 upper=3.141592653589793 effort=4.0 velocity=4.0
- joint front_left_upper_leg_rev_joint: limit lower=0.0 upper=1.9198621771937625 effort=4.0 velocity=4.0 -> lower=-3.141592653589793 upper=3.141592653589793 effort=4.0 velocity=4.0
- joint front_right_hip_rev_joint: axis 1 0 0 -> -1 0 0
- joint front_right_lower_leg_rev_joint: axis 0 1 0 -> 0 -1 0; limit lower=-1.3962634015954636 upper=1.038470904936626 effort=4.0 velocity=4.0 -> lower=-3.141592653589793 upper=3.141592653589793 effort=4.0 velocity=4.0
- joint front_right_upper_leg_rev_joint: limit lower=0.0 upper=1.9198621771937625 effort=4.0 velocity=4.0 -> lower=-3.141592653589793 upper=3.141592653589793 effort=4.0 velocity=4.0

File: quad_ws/src/quad_udrf/urdf/zuko.urdf.xacro (robot description, xacro)
@@ -110,5 +110,5 @@
 		height="0"
 		matname="brown"
-		meshfile="package://stl/center_front.stl"
+		meshfile="package://quad_urdf/stl/center_front.stl"
 		meshscale="1 1 1" />
 	<xacro:mesh_link name="side_left_link"
@@ -123,5 +123,5 @@
 		height="0"
 		matname="brown"
-		meshfile="package://stl/side_left.stl"
+		meshfile="package://quad_urdf/stl/side_left.stl"
 		meshscale="1 1 1" />
 	<xacro:mesh_link name="side_right_link"
@@ -136,5 +136,5 @@
 		height="0"
 		matname="brown"
-		meshfile="package://stl/side_right.stl"
+		meshfile="package://quad_urdf/stl/side_right.stl"
 		meshscale="1 1 1" />
 	<xacro:mesh_link name="center_back_link"
@@ -149,5 +149,5 @@
 		height="0"
 		matname="brown"
-		meshfile="package://stl/center_back.stl"
+		meshfile="package://quad_urdf/stl/center_back.stl"
 		meshscale="1 1 1" />
 	<xacro:mesh_link name="bridge_front_link"
@@ -162,5 +162,5 @@
 		height="0"
 		matname="white"
-		meshfile="package://stl/bridge_front.stl"
+		meshfile="package://quad_urdf/quad_urdf/stl/bridge_front.stl"
 		meshscale="1 1 1" />
 	<xacro:mesh_link name="bridge_back_link"
@@ -175,5 +175,5 @@
 		height="0"
 		matname="white"
-		meshfile="package://stl/bridge_back.stl"
+		meshfile="package://quad_urdf/stl/bridge_back.stl"
 		meshscale="1 1 1" />
 	<xacro:mesh_link name="face_link"
@@ -188,5 +188,5 @@
 		height="0"
 		matname="brown"
-		meshfile="package://stl/face.stl"
+		meshfile="package://quad_urdf/stl/face.stl"
 		meshscale="1 1 1" />
 	<xacro:mesh_link name="butt_link"
@@ -201,5 +201,5 @@
 		height="0"
 		matname="brown"
-		meshfile="package://stl/butt.stl"
+		meshfile="package://quad_urdf/stl/butt.stl"
 		meshscale="1 1 1" />
 <!-- STATIC Joints -->
@@ -279,5 +279,5 @@
 				height="0"
 				matname="white"
-				meshfile="package://stl/hip_front.stl"
+				meshfile="package://quad_urdf/stl/hip_front.stl"
 				meshscale="1 1 1" />
 		<xacro:rev_joint name="front_left_hip_rev_joint"
@@ -305,5 +305,5 @@
 					height="0"
 					matname="brown"
-					meshfile="package://stl/upper_leg.stl"
+					meshfile="package://quad_urdf/stl/upper_leg.stl"
 					meshscale="1 1 1" />
 		<xacro:rev_joint name="front_left_upper_leg_rev_joint"
@@ -331,5 +331,5 @@
 					height="0"
 					matname="brown"
-					meshfile="package://stl/lower_leg.stl"
+					meshfile="package://quad_urdf/stl/lower_leg.stl"
 					meshscale="1 1 1" />
 		<xacro:rev_joint name="front_left_lower_leg_rev_joint"
@@ -358,5 +358,5 @@
 				height="0"
 				matname="white"
-				meshfile="package://stl/hip_front.stl"
+				meshfile="package://quad_urdf/stl/hip_front.stl"
 				meshscale="1 -1 1" />
 		<xacro:rev_joint name="front_right_hip_rev_joint"
@@ -384,5 +384,5 @@
 					height="0"
 					matname="brown"
-					meshfile="package://stl/upper_leg.stl"
+					meshfile="package://quad_urdf/stl/upper_leg.stl"
 					meshscale="1 1 1" />
 		<xacro:rev_joint name="front_right_upper_leg_rev_joint"
@@ -410,5 +410,5 @@
 					height="0"
 					matname="brown"
-					meshfile="package://stl/lower_leg.stl"
+					meshfile="package://quad_urdf/stl/lower_leg.stl"
 					meshscale="1 1 -1" />
 		<xacro:rev_joint name="front_right_lower_leg_rev_joint"
@@ -437,5 +437,5 @@
 				height="0"
 				matname="white"
-				meshfile="package://stl/hip_back.stl"
+				meshfile="package://quad_urdf/stl/hip_back.stl"
 				meshscale="1 1 1" />
 		<xacro:rev_joint name="back_left_hip_rev_joint"
@@ -463,5 +463,5 @@
 					height="0"
 					matname="brown"
-					meshfile="package://stl/upper_leg.stl"
+					meshfile="package://quad_urdf/stl/upper_leg.stl"
 					meshscale="1 1 1" />
 		<xacro:rev_joint name="back_left_upper_leg_rev_joint"
@@ -489,5 +489,5 @@
 					height="0"
 					matname="brown"
-					meshfile="package://stl/lower_leg.stl"
+					meshfile="package://quad_urdf/stl/lower_leg.stl"
 					meshscale="1 1 1" />
 		<xacro:rev_joint name="back_left_lower_leg_rev_joint"
@@ -516,5 +516,5 @@
 				height="0"
 				matname="white"
-				meshfile="package://stl/hip_back.stl"
+				meshfile="package://quad_urdf/stl/hip_back.stl"
 				meshscale="1 -1 1" />
 		<xacro:rev_joint name="back_right_hip_rev_joint"
@@ -542,5 +542,5 @@
 					height="0"
 					matname="brown"
-					meshfile="package://stl/upper_leg.stl"
+					meshfile="package://quad_urdf/stl/upper_leg.stl"
 					meshscale="1 1 1" />
 		<xacro:rev_joint name="back_right_upper_leg_rev_joint"
@@ -568,5 +568,5 @@
 					height="0.25"
 					matname="brown"
-					meshfile="package://stl/lower_leg.stl"
+					meshfile="package://quad_urdf/stl/lower_leg.stl"
 					meshscale="1 1 -1" />
 		<xacro:rev_joint name="back_right_lower_leg_rev_joint"
