Commit message: moved quad_urdf into quad_simulation

File: quad_ws/src/quad_simulation/quad_simulation/urdf/zuko.urdf (robot description, URDF)
Before this commit: robot zuko, 20 links, 19 joints
Links:
- added link battery_cover_link, mass 0.6; collision mesh filename=package://stl/battery_cover.stl scale=1 1 1; visual mesh filename=package://stl/battery_cover.stl scale=1 1 1
- added link electronics_cover_link, mass 0.6; collision mesh filename=package://stl/electronics_cover.stl scale=1 1 1; visual mesh filename=package://stl/electronics_cover.stl scale=1 1 1
- added link tail_link, mass 0.6; collision mesh filename=package://stl/tail.stl scale=1 1 1; visual mesh filename=package://stl/tail.stl scale=1 1 1
Joints:
- added joint battery_cover_joint: type fixed, parent base_link, child battery_cover_link, origin xyz=-0.09375 0 -0.039 rpy=3.141592653589793 0 3.141592653589793
- added joint electronics_cover_joint: type fixed, parent base_link, child electronics_cover_link, origin xyz=-0.092 0 0.019 rpy=0 0 3.141592653589793
- added joint tail_joint: type fixed, parent butt_link, child tail_link, origin xyz=-0.012419 0 0.025687 rpy=0 0 0 
- joint bridge_back_joint: origin xyz=0 0 -0.011 rpy=0 0 0 -> xyz=0 0 -0.010 rpy=0 0 0
- joint bridge_front_joint: origin xyz=0.0535 0 -0.011 rpy=0 0  0 -> xyz=0.0535 0 -0.010 rpy=0 0  0
- joint center_back_joint: origin xyz=-0.16599999999999998 0 0 rpy=0 0 0 -> xyz=-0.18399999999999997 0 0 rpy=0 0 0

File: quad_ws/src/quad_simulation/quad_simulation/urdf/zuko.urdf.xacro (robot description, xacro)
@@ -39,6 +39,6 @@
 		  <material>Gazebo/Black</material>
 		</xacro:if>
-		<xacro:if value="${matname == 'orange'}">
-		  <material>Gazebo/Orange</material>
+		<xacro:if value="${matname == 'white'}">
+		  <material>Gazebo/White</material>
 		</xacro:if>
 	</gazebo>
@@ -112,5 +112,5 @@
 		height="0"
 		matname="brown"
-		meshfile="package://quad_urdf/stl/center_front.stl"
+		meshfile="package://stl/center_front.stl"
 		meshscale="1 1 1" />
 	<xacro:mesh_link name="side_left_link"
@@ -125,5 +125,5 @@
 		height="0"
 		matname="brown"
-		meshfile="package://quad_urdf/stl/side_left.stl"
+		meshfile="package://stl/side_left.stl"
 		meshscale="1 1 1" />
 	<xacro:mesh_link name="side_right_link"
@@ -138,5 +138,5 @@
 		height="0"
 		matname="brown"
-		meshfile="package://quad_urdf/stl/side_right.stl"
+		meshfile="package://stl/side_right.stl"
 		meshscale="1 1 1" />
 	<xacro:mesh_link name="center_back_link"
@@ -151,5 +151,5 @@
 		height="0"
 		matname="brown"
-		meshfile="package://quad_urdf/stl/center_back.stl"
+		meshfile="package://stl/center_back.stl"
 		meshscale="1 1 1" />
 	<xacro:mesh_link name="bridge_front_link"
@@ -164,5 +164,5 @@
 		height="0"
 		matname="white"
-		meshfile="package://quad_urdf/stl/bridge_front.stl"
+		meshfile="package://stl/bridge_front.stl"
 		meshscale="1 1 1" />
 	<xacro:mesh_link name="bridge_back_link"
@@ -177,5 +177,5 @@
 		height="0"
 		matname="white"
-		meshfile="package://quad_urdf/stl/bridge_back.stl"
+		meshfile="package://stl/bridge_back.stl"
 		meshscale="1 1 1" />
 	<xacro:mesh_link name="face_link"
@@ -190,5 +190,5 @@
 		height="0"
 		matname="brown"
-		meshfile="package://quad_urdf/stl/face.stl"
+		meshfile="package://stl/face.stl"
 		meshscale="1 1 1" />
 	<xacro:mesh_link name="butt_link"
@@ -203,5 +203,5 @@
 		height="0"
 		matname="brown"
-		meshfile="package://quad_urdf/stl/butt.stl"
+		meshfile="package://stl/butt.stl"
 		meshscale="1 1 1" />
 	<xacro:mesh_link name="electronics_cover_link"
@@ -216,5 +216,5 @@
 		height="0"
 		matname="brown"
-		meshfile="package://quad_urdf/stl/electronics_cover.stl"
+		meshfile="package://stl/electronics_cover.stl"
 		meshscale="1 1 1" />
 	<xacro:mesh_link name="battery_cover_link"
@@ -229,5 +229,5 @@
 		height="0"
 		matname="brown"
-		meshfile="package://quad_urdf/stl/battery_cover.stl"
+		meshfile="package://stl/battery_cover.stl"
 		meshscale="1 1 1" />
 	<xacro:mesh_link name="tail_link"
@@ -242,5 +242,5 @@
 		height="0"
 		matname="white"
-		meshfile="package://quad_urdf/stl/tail.stl"
+		meshfile="package://stl/tail.stl"
 		meshscale="1 1 1" />
 <!-- STATIC Joints -->
@@ -335,5 +335,5 @@
 				height="0"
 				matname="white"
-				meshfile="package://quad_urdf/stl/hip_front.stl"
+				meshfile="package://stl/hip_front.stl"
 				meshscale="1 1 1" />
 		<xacro:rev_joint name="front_left_hip_rev_joint"
@@ -361,5 +361,5 @@
 					height="0"
 					matname="brown"
-					meshfile="package://quad_urdf/stl/upper_leg.stl"
+					meshfile="package://stl/upper_leg.stl"
 					meshscale="1 1 1" />
 		<xacro:rev_joint name="front_left_upper_leg_rev_joint"
@@ -387,5 +387,5 @@
 					height="0"
 					matname="brown"
-					meshfile="package://quad_urdf/stl/lower_leg.stl"
+					meshfile="package://stl/lower_leg.stl"
 					meshscale="1 1 1" />
 		<xacro:rev_joint name="front_left_lower_leg_rev_joint"
@@ -414,5 +414,5 @@
 				height="0"
 				matname="white"
-				meshfile="package://quad_urdf/stl/hip_front.stl"
+				meshfile="package://stl/hip_front.stl"
 				meshscale="1 -1 1" />
 		<xacro:rev_joint name="front_right_hip_rev_joint"
@@ -440,5 +440,5 @@
 					height="0"
 					matname="brown"
-					meshfile="package://quad_urdf/stl/upper_leg.stl"
+					meshfile="package://stl/upper_leg.stl"
 					meshscale="1 1 1" />
 		<xacro:rev_joint name="front_right_upper_leg_rev_joint"
@@ -466,5 +466,5 @@
 					height="0"
 					matname="brown"
-					meshfile="package://quad_urdf/stl/lower_leg.stl"
+					meshfile="package://stl/lower_leg.stl"
 					meshscale="1 1 -1" />
 		<xacro:rev_joint name="front_right_lower_leg_rev_joint"
@@ -493,5 +493,5 @@
 				height="0"
 				matname="white"
-				meshfile="package://quad_urdf/stl/hip_back.stl"
+				meshfile="package://stl/hip_back.stl"
 				meshscale="1 1 1" />
 		<xacro:rev_joint name="back_left_hip_rev_joint"
@@ -519,5 +519,5 @@
 					height="0"
 					matname="brown"
-					meshfile="package://quad_urdf/stl/upper_leg.stl"
+					meshfile="package://stl/upper_leg.stl"
 					meshscale="1 1 1" />
 		<xacro:rev_joint name="back_left_upper_leg_rev_joint"
@@ -545,5 +545,5 @@
 					height="0"
 					matname="brown"
-					meshfile="package://quad_urdf/stl/lower_leg.stl"
+					meshfile="package://stl/lower_leg.stl"
 					meshscale="1 1 1" />
 		<xacro:rev_joint name="back_left_lower_leg_rev_joint"
@@ -572,5 +572,5 @@
 				height="0"
 				matname="white"
-				meshfile="package://quad_urdf/stl/hip_back.stl"
+				meshfile="package://stl/hip_back.stl"
 				meshscale="1 -1 1" />
 		<xacro:rev_joint name="back_right_hip_rev_joint"
@@ -598,5 +598,5 @@
 					height="0"
 					matname="brown"
-					meshfile="package://quad_urdf/stl/upper_leg.stl"
+					meshfile="package://stl/upper_leg.stl"
 					meshscale="1 1 1" />
 		<xacro:rev_joint name="back_right_upper_leg_rev_joint"
@@ -624,5 +624,5 @@
 					height="0.25"
 					matname="brown"
-					meshfile="package://quad_urdf/stl/lower_leg.stl"
+					meshfile="package://stl/lower_leg.stl"
 					meshscale="1 1 -1" />
 		<xacro:rev_joint name="back_right_lower_leg_rev_joint"

Commit message: removed unneeded mesh collisions in URDF

File: quad_ws/src/quad_simulation/quad_simulation/urdf/zuko.urdf (robot description, URDF)
Before this commit: robot zuko, 23 links, 22 joints
Links:
- link back_left_hip_link: geometry collision box size=0 0 0; visual mesh filename=package://stl/hip_back.stl scale=1 1 1
- link back_left_upper_leg_link: geometry collision box size=0 0 0; visual mesh filename=package://stl/upper_leg.stl scale=1 1 1
- link back_right_hip_link: geometry collision box size=0 0 0; visual mesh filename=package://stl/hip_back.stl scale=1 -1 1
- link back_right_upper_leg_link: geometry collision box size=0 0 0; visual mesh filename=package://stl/upper_leg.stl scale=1 1 1
- link base_link: geometry collision box size=0 0 0; visual mesh filename=package://stl/center_front.stl scale=1 1 1
- link battery_cover_link: geometry collision box size=0 0 0; visual mesh filename=package://stl/battery_cover.stl scale=1 1 1
- link bridge_back_link: geometry collision box size=0 0 0; visual mesh filename=package://stl/bridge_back.stl scale=1 1 1
- link bridge_front_link: geometry collision box size=0 0 0; visual mesh filename=package://stl/bridge_front.stl scale=1 1 1
- link butt_link: geometry collision box size=0 0 0; visual mesh filename=package://stl/butt.stl scale=1 1 1
- link center_back_link: geometry collision box size=0 0 0; visual mesh filename=package://stl/center_back.stl scale=1 1 1
- link electronics_cover_link: geometry collision box size=0 0 0; visual mesh filename=package://stl/electronics_cover.stl scale=1 1 1
- link face_link: geometry collision box size=0 0 0; visual mesh filename=package://stl/face.stl scale=1 1 1
- link front_left_hip_link: geometry collision box size=0 0 0; visual mesh filename=package://stl/hip_front.stl scale=1 1 1
- link front_left_upper_leg_link: geometry collision box size=0 0 0; visual mesh filename=package://stl/upper_leg.stl scale=1 1 1
- link front_right_hip_link: geometry collision box size=0 0 0; visual mesh filename=package://stl/hip_front.stl scale=1 -1 1
- link front_right_upper_leg_link: geometry collision box size=0 0 0; visual mesh filename=package://stl/upper_leg.stl scale=1 1 1
- link side_left_link: geometry collision box size=0 0 0; visual mesh filename=package://stl/side_left.stl scale=1 1 1
- link side_right_link: geometry collision box size=0 0 0; visual mesh filename=package://stl/side_right.stl scale=1 1 1
- link tail_link: geometry collision box size=0 0 0; visual mesh filename=package://stl/tail.stl scale=1 1 1

File: quad_ws/src/quad_simulation/quad_simulation/urdf/zuko.urdf.xacro (robot description, xacro)
@@ -25,5 +25,34 @@
 		<origin rpy="${origin_rpy}" xyz="${c_xyz}" />
 		<geometry>
-		  <!--<box size="${length} ${width} ${height}" />-->
+		  <box size="${length} ${width} ${height}" />
+		</geometry>
+	  </collision>
+	  <inertial>
+		<mass value="${mass}" />
+		<origin rpy="${i_rpy}" xyz="${i_xyz}" /> <!-- Inertial Axes -->
+		<inertia ixx="${mass * (width * width + height * height)/12.0}" ixy="${0}" ixz="${0}" iyx="${0}" iyy="${mass * (length * length + height * height)/12.0}" iyz="${0}" izx="${0}" izy="${0}" izz="${mass * (length * length + width * width)/12.0}" />
+	  </inertial>
+	</link>
+	<gazebo reference="${name}">
+		<xacro:if value="${matname == 'black'}">
+		  <material>Gazebo/Black</material>
+		</xacro:if>
+		<xacro:if value="${matname == 'white'}">
+		  <material>Gazebo/White</material>
+		</xacro:if>
+	</gazebo>
+</xacro:macro>
+<xacro:macro name="mesh_mesh_link" params="name origin_xyz origin_rpy meshfile meshscale c_xyz matname mass i_xyz i_rpy length width height">
+	<link name="${name}">
+	  <visual>
+		<origin rpy="${origin_rpy}" xyz="${origin_xyz}" />
+		<geometry>
+		  <mesh filename="${meshfile}" scale="${meshscale}"/>
+		</geometry>
+		<material name="${matname}"/>
+	  </visual>
+	  <collision>
+		<origin rpy="${origin_rpy}" xyz="${c_xyz}" />
+		<geometry>
 		  <mesh filename="${meshfile}" scale="${meshscale}"/>
 		</geometry>
@@ -376,5 +405,5 @@
 				    parent="front_left_hip_link"
 				    child="front_left_upper_leg_link" />
-		<xacro:mesh_link name="front_left_lower_leg_link"
+		<xacro:mesh_mesh_link name="front_left_lower_leg_link"
 					origin_rpy="${pi/2} ${pi/2} ${pi}"
 					origin_xyz="0 -${upper_leg_origin_offset_to_center_of_leg} 0"
@@ -455,5 +484,5 @@
 				    parent="front_right_hip_link"
 				    child="front_right_upper_leg_link" />
-		<xacro:mesh_link name="front_right_lower_leg_link"
+		<xacro:mesh_mesh_link name="front_right_lower_leg_link"
 					origin_rpy="${pi/2} ${pi/2}  ${pi}"
 					origin_xyz="0 ${upper_leg_origin_offset_to_center_of_leg} 0"
@@ -534,5 +563,5 @@
 				    parent="back_left_hip_link"
 				    child="back_left_upper_leg_link" />
-		<xacro:mesh_link name="back_left_lower_leg_link"
+		<xacro:mesh_mesh_link name="back_left_lower_leg_link"
 					origin_rpy="${pi/2} ${pi/2} ${pi}"
 					origin_xyz="0 -${upper_leg_origin_offset_to_center_of_leg} 0"
@@ -613,5 +642,5 @@
 				    parent="back_right_hip_link"
 				    child="back_right_upper_leg_link" />
-		<xacro:mesh_link name="back_right_lower_leg_link"
+		<xacro:mesh_mesh_link name="back_right_lower_leg_link"
 					origin_rpy="${pi/2} ${pi/2} ${pi}"
 					origin_xyz="0 ${upper_leg_origin_offset_to_center_of_leg} 0"
