Commit message: URDF update

File: quad_ws/src/quad_udrf/urdf/zuko.urdf.xacro (robot description, xacro)
@@ -95,15 +95,17 @@
 <!-- STATIC Links -->
 	<!-- Offsets-->
+	<!-- center front and center back orgin is 2.5mm inside the part-->
 	<xacro:property name="center_thickness" value="0.018" />
 	<xacro:property name="center_orgin_offset" value="0.0025" />
 	<xacro:property name="side_length" value="0.148" />
 	<xacro:property name="bridge_length" value="0.0535" />
+	<xacro:property name="center_origin_to_top_cover_inset" value="0.019" />
 	<xacro:mesh_link name="base_link"
 		origin_rpy="${pi/2} 0 -${pi/2}"
-		origin_xyz="-${center_orgin_offset} 0 0"
-		i_rpy="0 0 0"
-		i_xyz="0 0 0"
-		mass="0.6"
-		c_xyz="0 0 0"
+		origin_xyz="${-center_orgin_offset} 0 0"
+		i_rpy="0 0 0"
+		i_xyz="0 0 0"
+		mass="0.6"
+		c_xyz="${-center_orgin_offset} 0 0"
 		length="0"
 		width="0"
@@ -144,5 +146,5 @@
 		i_xyz="0 0 0"
 		mass="0.6"
-		c_xyz="0 0 0"
+		c_xyz="${center_orgin_offset} 0 0"
 		length="0"
 		width="0"
@@ -162,5 +164,5 @@
 		height="0"
 		matname="white"
-		meshfile="package://quad_urdf/quad_urdf/stl/bridge_front.stl"
+		meshfile="package://quad_urdf/stl/bridge_front.stl"
 		meshscale="1 1 1" />
 	<xacro:mesh_link name="bridge_back_link"
@@ -203,9 +205,48 @@
 		meshfile="package://quad_urdf/stl/butt.stl"
 		meshscale="1 1 1" />
+	<xacro:mesh_link name="electronics_cover_link"
+		origin_rpy="0 0 0"
+		origin_xyz="0 0 0"
+		i_rpy="0 0 0"
+		i_xyz="0 0 0"
+		mass="0.6"
+		c_xyz="0 0 0"
+		length="0"
+		width="0"
+		height="0"
+		matname="brown"
+		meshfile="package://quad_urdf/stl/electronics_cover.stl"
+		meshscale="1 1 1" />
+	<xacro:mesh_link name="battery_cover_link"
+		origin_rpy="0 0 0"
+		origin_xyz="0 0 0"
+		i_rpy="0 0 0"
+		i_xyz="0 0 0"
+		mass="0.6"
+		c_xyz="0 0 0"
+		length="0"
+		width="0"
+		height="0"
+		matname="brown"
+		meshfile="package://quad_urdf/stl/battery_cover.stl"
+		meshscale="1 1 1" />
+	<xacro:mesh_link name="tail_link"
+		origin_rpy="${pi/2} ${35 * pi/180} 0"
+		origin_xyz="0 0 0"
+		i_rpy="0 0 0"
+		i_xyz="0 0 0"
+		mass="0.6"
+		c_xyz="0 0 0"
+		length="0"
+		width="0"
+		height="0"
+		matname="white"
+		meshfile="package://quad_urdf/stl/tail.stl"
+		meshscale="1 1 1" />
 <!-- STATIC Joints -->
 <xacro:frame_joint name="side_left_joint"
 			type="fixed"
 			origin_rpy="0 0 0"
-			origin_xyz="-${center_thickness + side_length} 0.060 0.015"
+			origin_xyz="${-center_thickness - side_length} 0.060 0.015"
 			parent="base_link"
 			child="side_left_link"/>
@@ -219,5 +260,5 @@
 			type="fixed"
 			origin_rpy="0 0 0"
-			origin_xyz="-${side_length + center_thickness} 0 0"
+			origin_xyz="${-side_length - center_thickness - center_thickness} 0 0"
 			parent="base_link"
 			child="center_back_link"/>
@@ -225,5 +266,5 @@
 			type="fixed"
 			origin_rpy="0 0  0"
-			origin_xyz="${bridge_length} 0 -0.011"
+			origin_xyz="${bridge_length} 0 -0.010"
 			parent="base_link"
 			child="bridge_front_link"/>
@@ -231,5 +272,5 @@
 			type="fixed"
 			origin_rpy="0 0 0"
-			origin_xyz="0 0 -0.011"
+			origin_xyz="0 0 -0.010"
 			parent="center_back_link"
 			child="bridge_back_link"/>
@@ -246,4 +287,22 @@
 			parent="bridge_back_link"
 			child="butt_link"/>
+<xacro:frame_joint name="electronics_cover_joint"
+			type="fixed"
+			origin_rpy="0 0 ${pi}"
+			origin_xyz="${-0.089 - 0.003} 0 ${center_origin_to_top_cover_inset}"
+			parent="base_link"
+			child="electronics_cover_link"/>
+<xacro:frame_joint name="battery_cover_joint"
+			type="fixed"
+			origin_rpy="${pi} 0 ${pi}"
+			origin_xyz="${-0.09075 - 0.003} 0 -0.039"
+			parent="base_link"
+			child="battery_cover_link"/>
+<xacro:frame_joint name="tail_joint"
+			type="fixed"
+			origin_rpy="0 0 0 "
+			origin_xyz="-0.012419 0 0.025687"
+			parent="butt_link"
+			child="tail_link"/>
 <!-- Hips/Legs Links/Joints -->
 	<!-- Offsets -->
@@ -264,7 +323,4 @@
 		<xacro:property name="lower_leg_upper_limit" value="${180 * pi/180}" />
 		<xacro:property name="lower_leg_lower_limit" value="${-180 * pi/180}" />
-<!--
-<xacro:property name="path" value="package://stl" />
--->
 	<!-- FRONT LEFT -->
 		<xacro:mesh_link name="front_left_hip_link"
@@ -583,9 +639,10 @@
 				    parent="back_right_upper_leg_link"
 				    child="back_right_lower_leg_link" />
+<!-- GAZEBO related requirements-->
 <!--
-<xacro:transmission leg="front_left"/>
-<xacro:transmission leg="front_right"/>
-<xacro:transmission leg="back_left"/>
-<xacro:transmission leg="back_right"/>
+	<xacro:transmission leg="front_left"/>
+	<xacro:transmission leg="front_right"/>
+	<xacro:transmission leg="back_left"/>
+	<xacro:transmission leg="back_right"/>
 -->
 </robot>

Commit message: brought back quad_urdf into separate package for seperation of concerns

File: quad_ws/src/quad_udrf/urdf/zuko.urdf.xacro (robot description, xacro)
@@ -25,34 +25,5 @@
 		<origin rpy="${origin_rpy}" xyz="${c_xyz}" />
 		<geometry>
-		  <box size="${length} ${width} ${height}" />
-		</geometry>
-	  </collision>
-	  <inertial>
-		<mass value="${mass}" />
-		<origin rpy="${i_rpy}" xyz="${i_xyz}" /> <!-- Inertial Axes -->
-		<inertia ixx="${mass * (width * width + height * height)/12.0}" ixy="${0}" ixz="${0}" iyx="${0}" iyy="${mass * (length * length + height * height)/12.0}" iyz="${0}" izx="${0}" izy="${0}" izz="${mass * (length * length + width * width)/12.0}" />
-	  </inertial>
-	</link>
-	<gazebo reference="${name}">
-		<xacro:if value="${matname == 'black'}">
-		  <material>Gazebo/Black</material>
-		</xacro:if>
-		<xacro:if value="${matname == 'white'}">
-		  <material>Gazebo/White</material>
-		</xacro:if>
-	</gazebo>
-</xacro:macro>
-<xacro:macro name="mesh_mesh_link" params="name origin_xyz origin_rpy meshfile meshscale c_xyz matname mass i_xyz i_rpy length width height">
-	<link name="${name}">
-	  <visual>
-		<origin rpy="${origin_rpy}" xyz="${origin_xyz}" />
-		<geometry>
-		  <mesh filename="${meshfile}" scale="${meshscale}"/>
-		</geometry>
-		<material name="${matname}"/>
-	  </visual>
-	  <collision>
-		<origin rpy="${origin_rpy}" xyz="${c_xyz}" />
-		<geometry>
+		  <!--<box size="${length} ${width} ${height}" />-->
 		  <mesh filename="${meshfile}" scale="${meshscale}"/>
 		</geometry>
@@ -68,6 +39,6 @@
 		  <material>Gazebo/Black</material>
 		</xacro:if>
-		<xacro:if value="${matname == 'white'}">
-		  <material>Gazebo/White</material>
+		<xacro:if value="${matname == 'orange'}">
+		  <material>Gazebo/Orange</material>
 		</xacro:if>
 	</gazebo>
@@ -124,7 +95,5 @@
 <!-- STATIC Links -->
 	<!-- Offsets-->
-	<!-- center front and center back orgin is 2.5mm inside the part-->
 	<xacro:property name="center_thickness" value="0.018" />
-	<xacro:property name="center_orgin_offset" value="0.0025" />
 	<xacro:property name="side_length" value="0.148" />
 	<xacro:property name="bridge_length" value="0.0535" />
@@ -132,14 +101,14 @@
 	<xacro:mesh_link name="base_link"
 		origin_rpy="${pi/2} 0 -${pi/2}"
-		origin_xyz="${-center_orgin_offset} 0 0"
-		i_rpy="0 0 0"
-		i_xyz="0 0 0"
-		mass="0.6"
-		c_xyz="${-center_orgin_offset} 0 0"
-		length="0"
-		width="0"
-		height="0"
-		matname="brown"
-		meshfile="package://stl/center_front.stl"
+		origin_xyz="0 0 0"
+		i_rpy="0 0 0"
+		i_xyz="0 0 0"
+		mass="0.6"
+		c_xyz="0 0 0"
+		length="0"
+		width="0"
+		height="0"
+		matname="brown"
+		meshfile="package://quad_urdf/stl/center_front.stl"
 		meshscale="1 1 1" />
 	<xacro:mesh_link name="side_left_link"
@@ -154,5 +123,5 @@
 		height="0"
 		matname="brown"
-		meshfile="package://stl/side_left.stl"
+		meshfile="package://quad_urdf/stl/side_left.stl"
 		meshscale="1 1 1" />
 	<xacro:mesh_link name="side_right_link"
@@ -167,18 +136,18 @@
 		height="0"
 		matname="brown"
-		meshfile="package://stl/side_right.stl"
+		meshfile="package://quad_urdf/stl/side_right.stl"
 		meshscale="1 1 1" />
 	<xacro:mesh_link name="center_back_link"
 		origin_rpy="${pi/2} 0 ${pi/2}"
-		origin_xyz="${center_orgin_offset} 0 0"
-		i_rpy="0 0 0"
-		i_xyz="0 0 0"
-		mass="0.6"
-		c_xyz="${center_orgin_offset} 0 0"
-		length="0"
-		width="0"
-		height="0"
-		matname="brown"
-		meshfile="package://stl/center_back.stl"
+		origin_xyz="0 0 0"
+		i_rpy="0 0 0"
+		i_xyz="0 0 0"
+		mass="0.6"
+		c_xyz="0 0 0"
+		length="0"
+		width="0"
+		height="0"
+		matname="brown"
+		meshfile="package://quad_urdf/stl/center_back.stl"
 		meshscale="1 1 1" />
 	<xacro:mesh_link name="bridge_front_link"
@@ -193,5 +162,5 @@
 		height="0"
 		matname="white"
-		meshfile="package://stl/bridge_front.stl"
+		meshfile="package://quad_urdf/stl/bridge_front.stl"
 		meshscale="1 1 1" />
 	<xacro:mesh_link name="bridge_back_link"
@@ -206,5 +175,5 @@
 		height="0"
 		matname="white"
-		meshfile="package://stl/bridge_back.stl"
+		meshfile="package://quad_urdf/stl/bridge_back.stl"
 		meshscale="1 1 1" />
 	<xacro:mesh_link name="face_link"
@@ -219,5 +188,5 @@
 		height="0"
 		matname="brown"
-		meshfile="package://stl/face.stl"
+		meshfile="package://quad_urdf/stl/face.stl"
 		meshscale="1 1 1" />
 	<xacro:mesh_link name="butt_link"
@@ -232,5 +201,5 @@
 		height="0"
 		matname="brown"
-		meshfile="package://stl/butt.stl"
+		meshfile="package://quad_urdf/stl/butt.stl"
 		meshscale="1 1 1" />
 	<xacro:mesh_link name="electronics_cover_link"
@@ -245,5 +214,5 @@
 		height="0"
 		matname="brown"
-		meshfile="package://stl/electronics_cover.stl"
+		meshfile="package://quad_urdf/stl/electronics_cover.stl"
 		meshscale="1 1 1" />
 	<xacro:mesh_link name="battery_cover_link"
@@ -258,5 +227,5 @@
 		height="0"
 		matname="brown"
-		meshfile="package://stl/battery_cover.stl"
+		meshfile="package://quad_urdf/stl/battery_cover.stl"
 		meshscale="1 1 1" />
 	<xacro:mesh_link name="tail_link"
@@ -271,5 +240,5 @@
 		height="0"
 		matname="white"
-		meshfile="package://stl/tail.stl"
+		meshfile="package://quad_urdf/stl/tail.stl"
 		meshscale="1 1 1" />
 <!-- STATIC Joints -->
@@ -364,5 +333,5 @@
 				height="0"
 				matname="white"
-				meshfile="package://stl/hip_front.stl"
+				meshfile="package://quad_urdf/stl/hip_front.stl"
 				meshscale="1 1 1" />
 		<xacro:rev_joint name="front_left_hip_rev_joint"
@@ -390,5 +359,5 @@
 					height="0"
 					matname="brown"
-					meshfile="package://stl/upper_leg.stl"
+					meshfile="package://quad_urdf/stl/upper_leg.stl"
 					meshscale="1 1 1" />
 		<xacro:rev_joint name="front_left_upper_leg_rev_joint"
@@ -405,5 +374,5 @@
 				    parent="front_left_hip_link"
 				    child="front_left_upper_leg_link" />
-		<xacro:mesh_mesh_link name="front_left_lower_leg_link"
+		<xacro:mesh_link name="front_left_lower_leg_link"
 					origin_rpy="${pi/2} ${pi/2} ${pi}"
 					origin_xyz="0 -${upper_leg_origin_offset_to_center_of_leg} 0"
@@ -416,5 +385,5 @@
 					height="0"
 					matname="brown"
-					meshfile="package://stl/lower_leg.stl"
+					meshfile="package://quad_urdf/stl/lower_leg.stl"
 					meshscale="1 1 1" />
 		<xacro:rev_joint name="front_left_lower_leg_rev_joint"
@@ -443,5 +412,5 @@
 				height="0"
 				matname="white"
-				meshfile="package://stl/hip_front.stl"
+				meshfile="package://quad_urdf/stl/hip_front.stl"
 				meshscale="1 -1 1" />
 		<xacro:rev_joint name="front_right_hip_rev_joint"
@@ -469,5 +438,5 @@
 					height="0"
 					matname="brown"
-					meshfile="package://stl/upper_leg.stl"
+					meshfile="package://quad_urdf/stl/upper_leg.stl"
 					meshscale="1 1 1" />
 		<xacro:rev_joint name="front_right_upper_leg_rev_joint"
@@ -484,5 +453,5 @@
 				    parent="front_right_hip_link"
 				    child="front_right_upper_leg_link" />
-		<xacro:mesh_mesh_link name="front_right_lower_leg_link"
+		<xacro:mesh_link name="front_right_lower_leg_link"
 					origin_rpy="${pi/2} ${pi/2}  ${pi}"
 					origin_xyz="0 ${upper_leg_origin_offset_to_center_of_leg} 0"
@@ -495,5 +464,5 @@
 					height="0"
 					matname="brown"
-					meshfile="package://stl/lower_leg.stl"
+					meshfile="package://quad_urdf/stl/lower_leg.stl"
 					meshscale="1 1 -1" />
 		<xacro:rev_joint name="front_right_lower_leg_rev_joint"
@@ -522,5 +491,5 @@
 				height="0"
 				matname="white"
-				meshfile="package://stl/hip_back.stl"
+				meshfile="package://quad_urdf/stl/hip_back.stl"
 				meshscale="1 1 1" />
 		<xacro:rev_joint name="back_left_hip_rev_joint"
@@ -548,5 +517,5 @@
 					height="0"
 					matname="brown"
-					meshfile="package://stl/upper_leg.stl"
+					meshfile="package://quad_urdf/stl/upper_leg.stl"
 					meshscale="1 1 1" />
 		<xacro:rev_joint name="back_left_upper_leg_rev_joint"
@@ -563,5 +532,5 @@
 				    parent="back_left_hip_link"
 				    child="back_left_upper_leg_link" />
-		<xacro:mesh_mesh_link name="back_left_lower_leg_link"
+		<xacro:mesh_link name="back_left_lower_leg_link"
 					origin_rpy="${pi/2} ${pi/2} ${pi}"
 					origin_xyz="0 -${upper_leg_origin_offset_to_center_of_leg} 0"
@@ -574,5 +543,5 @@
 					height="0"
 					matname="brown"
-					meshfile="package://stl/lower_leg.stl"
+					meshfile="package://quad_urdf/stl/lower_leg.stl"
 					meshscale="1 1 1" />
 		<xacro:rev_joint name="back_left_lower_leg_rev_joint"
@@ -601,5 +570,5 @@
 				height="0"
 				matname="white"
-				meshfile="package://stl/hip_back.stl"
+				meshfile="package://quad_urdf/stl/hip_back.stl"
 				meshscale="1 -1 1" />
 		<xacro:rev_joint name="back_right_hip_rev_joint"
@@ -627,5 +596,5 @@
 					height="0"
 					matname="brown"
-					meshfile="package://stl/upper_leg.stl"
+					meshfile="package://quad_urdf/stl/upper_leg.stl"
 					meshscale="1 1 1" />
 		<xacro:rev_joint name="back_right_upper_leg_rev_joint"
@@ -642,5 +611,5 @@
 				    parent="back_right_hip_link"
 				    child="back_right_upper_leg_link" />
-		<xacro:mesh_mesh_link name="back_right_lower_leg_link"
+		<xacro:mesh_link name="back_right_lower_leg_link"
 					origin_rpy="${pi/2} ${pi/2} ${pi}"
 					origin_xyz="0 ${upper_leg_origin_offset_to_center_of_leg} 0"
@@ -653,5 +622,5 @@
 					height="0.25"
 					matname="brown"
-					meshfile="package://stl/lower_leg.stl"
+					meshfile="package://quad_urdf/stl/lower_leg.stl"
 					meshscale="1 1 -1" />
 		<xacro:rev_joint name="back_right_lower_leg_rev_joint"
